File: audio.kicad_sch (KiCad schematic)
At the start: 15 parts, among them J6 Audio Left, J7 Audio Right, J8 Stereo, U17 74LS08

Commit message: update page info
Other:
- company: (none) -> Dragon Data
Changed lines of the file:
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@@
 (kicad_sch (version 20230121) (generator eeschema)
-  (paper "A4")
+  (paper "A3")
+  (title_block
+    (date "2024-01-07")
+    (rev "3.0")
+    (company "Dragon Data")
+    (comment 1 "Modified by Julian Brown")
+    (comment 2 "SAMx4 by Ciaran Anscomb")
+  )
   (junction (at 207.518 37.338) (diameter 0) (color 0 0 0 0)
   )

Commit message: switch to fpga
Connections:
- net A0 renamed Z0
- net A1 renamed Z1
- net D0 renamed DC0
- net D1 renamed DC1
- net D2 renamed DC2
- net D3 renamed DC3
- net D4 renamed DC4
- net D5 renamed DC5
- net D6 renamed DC6
- net D7 renamed DC7
Other:
- moved on the sheet: J6, J7
