File: Dragon32.kicad_pcb (KiCad board)
At the start: 2 copper layers, 253 x 169.1 mm, 170 parts, among them IC1 LM393DR, IC10 74ACT138, IC11 74ACT244N, IC16 74ACT244N, IC19 MC6809E, IC24 74ACT244N, IC31 74ACT02, IC33 74ACT138N, IC34 CD4050BDR, J1 Video Output Female, J2 Board Interconnect Female, J3 Conn_02x08_Odd_Even, J4 JTAG, J5 6-bit DAC, J6 Audio Left, J7 Audio Right, J8 Stereo, SW1 RESET, U1 AS6C1008-TIN, U10 4052, U11 TS5A3166DBVR, U12 6551, U13 4069, U14 LM348DR, U17 74LS08, U2 AS6C1008-55TIN, U3 XC95144XL-TQ100, U4 TPS7A2433DBVR, U5 W65C21, U6 W65C21, U7 W65C21, U8 28C256, U9 74HCT1G08, X1 14.31818MHz, X2 1.8432MHz

Commit message: switch to fpga
Parts:
- removed D11, D12, D13, D14, D15, D16, D17: 1N914, Diode_SMD:D_SOD-323_HandSoldering
- removed IC11, IC16: 74ACT244N, Package_SO:SOIC-20W_7.5x12.8mm_P1.27mm
- removed JP6: ROM A14, Dragon:Jumper_4
- removed R13, R14, R40, R41, R54, R55: 4K7, Resistor_SMD:R_0805_2012Metric_Pad1.20x1.40mm_HandSolder
- removed R2, R20, R27, R4: 22R, Resistor_SMD:R_0805_2012Metric_Pad1.20x1.40mm_HandSolder
- removed R35, R37: 47R, Resistor_SMD:R_0805_2012Metric_Pad1.20x1.40mm_HandSolder
- removed R5: 100R, Resistor_SMD:R_0805_2012Metric_Pad1.20x1.40mm_HandSolder
- removed R57, R58: 47K, Resistor_SMD:R_0805_2012Metric_Pad1.20x1.40mm_HandSolder
- removed R59, R60: 100K, Resistor_SMD:R_0805_2012Metric_Pad1.20x1.40mm_HandSolder
- removed REG1: LM79L05_TO92, Package_TO_SOT_SMD:SOT-89-3_Handsoldering
- removed RN1, RN2: 22R, Package_SO:SOIC-16_3.9x9.9mm_P1.27mm
- removed X1: 14.31818MHz, Oscillator:Oscillator_SMD_ECS_2520MV-xxx-xx-4Pin_2.5x2.0mm
- added C20: 10u, Capacitor_SMD:CP_Elec_5x5.3, F.Cu at (112.3, 62.0)
- added C21: 10u, Capacitor_SMD:CP_Elec_5x5.3, F.Cu at (112.3, 70.4)
- added C24: 10u, Capacitor_SMD:CP_Elec_5x5.3, F.Cu at (118.1, 75.2)
- added C25: 0.1uF, Capacitor_SMD:C_0805_2012Metric_Pad1.18x1.45mm_HandSolder, F.Cu at (164.5, -50.0)
- added C28: 0.1uF, Capacitor_SMD:C_0805_2012Metric_Pad1.18x1.45mm_HandSolder, F.Cu at (164.5, -47.0)
- added C29: 4.7uF, Capacitor_SMD:C_0805_2012Metric_Pad1.18x1.45mm_HandSolder, F.Cu at (164.5, -44.0)
- added C34: 4.7uF, Capacitor_SMD:C_0805_2012Metric_Pad1.18x1.45mm_HandSolder, F.Cu at (164.5, -40.9)
- added C36: 0.47uF, Capacitor_SMD:C_0805_2012Metric_Pad1.18x1.45mm_HandSolder, F.Cu at (164.5, -37.9)
- added C37: 0.47uF, Capacitor_SMD:C_0805_2012Metric_Pad1.18x1.45mm_HandSolder, F.Cu at (169.4, -56.0)
- added C40: 0.47uF, Capacitor_SMD:C_0805_2012Metric_Pad1.18x1.45mm_HandSolder, F.Cu at (169.4, -53.0)
- added C41: 0.47uF, Capacitor_SMD:C_0805_2012Metric_Pad1.18x1.45mm_HandSolder, F.Cu at (169.4, -50.0)
- added C47: 4.7uF, Capacitor_SMD:C_0805_2012Metric_Pad1.18x1.45mm_HandSolder, F.Cu at (169.4, -47.0)
- added C49: 4.7uF, Capacitor_SMD:C_0805_2012Metric_Pad1.18x1.45mm_HandSolder, F.Cu at (169.4, -44.0)
- added C50: 0.47uF, Capacitor_SMD:C_0805_2012Metric_Pad1.18x1.45mm_HandSolder, F.Cu at (169.4, -40.9)
- added C52: 4.7uF, Capacitor_SMD:C_0805_2012Metric_Pad1.18x1.45mm_HandSolder, F.Cu at (169.4, -37.9)
- added C53: 4.7uF, Capacitor_SMD:C_0805_2012Metric_Pad1.18x1.45mm_HandSolder, F.Cu at (174.2, -56.0)
- added C54: 4.7uF, Capacitor_SMD:C_0805_2012Metric_Pad1.18x1.45mm_HandSolder, F.Cu at (174.2, -53.0)
- added C55: 1u, Capacitor_SMD:C_0805_2012Metric_Pad1.18x1.45mm_HandSolder, F.Cu at (174.2, -50.0)
- added C56: 4.7uF, Capacitor_SMD:C_0805_2012Metric_Pad1.18x1.45mm_HandSolder, F.Cu at (174.2, -47.0)
- added C57: 0.47uF, Capacitor_SMD:C_0805_2012Metric_Pad1.18x1.45mm_HandSolder, F.Cu at (174.2, -44.0)
- added C58: 1u, Capacitor_SMD:C_0805_2012Metric_Pad1.18x1.45mm_HandSolder, F.Cu at (174.2, -40.9)
- added C59: 4.7uF, Capacitor_SMD:C_0805_2012Metric_Pad1.18x1.45mm_HandSolder, F.Cu at (174.2, -37.9)
- added C60: 0.47uF, Capacitor_SMD:C_0805_2012Metric_Pad1.18x1.45mm_HandSolder, F.Cu at (179.0, -56.0)
- added C61: 1u, Capacitor_SMD:C_0805_2012Metric_Pad1.18x1.45mm_HandSolder, F.Cu at (179.0, -53.0)
- added C62: 1u, Capacitor_SMD:C_0805_2012Metric_Pad1.18x1.45mm_HandSolder, F.Cu at (179.0, -50.0)
- added C63: 0.01uF, Capacitor_SMD:C_0805_2012Metric_Pad1.18x1.45mm_HandSolder, F.Cu at (179.0, -47.0)
- added C64: 4.7uF, Capacitor_SMD:C_0805_2012Metric_Pad1.18x1.45mm_HandSolder, F.Cu at (179.0, -44.0)
- added C65: 4.7uF, Capacitor_SMD:C_0805_2012Metric_Pad1.18x1.45mm_HandSolder, F.Cu at (179.0, -40.9)
- added C66: 4.7uF, Capacitor_SMD:C_0805_2012Metric_Pad1.18x1.45mm_HandSolder, F.Cu at (179.0, -37.9)
- added C67: 4.7uF, Capacitor_SMD:C_0805_2012Metric_Pad1.18x1.45mm_HandSolder, F.Cu at (183.8, -56.0)
- added C70: 4.7uF, Capacitor_SMD:C_0805_2012Metric_Pad1.18x1.45mm_HandSolder, F.Cu at (183.8, -53.0)
- added C71: 0.47uF, Capacitor_SMD:C_0805_2012Metric_Pad1.18x1.45mm_HandSolder, F.Cu at (183.8, -50.0)
- added C72: 0.47uF, Capacitor_SMD:C_0805_2012Metric_Pad1.18x1.45mm_HandSolder, F.Cu at (183.8, -47.0)
- added C73: 0.47uF, Capacitor_SMD:C_0805_2012Metric_Pad1.18x1.45mm_HandSolder, F.Cu at (183.8, -44.0)
- added C74: 0.1uF, Capacitor_SMD:C_0805_2012Metric_Pad1.18x1.45mm_HandSolder, F.Cu at (183.8, -40.9)
- added C75: 0.1uF, Capacitor_SMD:C_0805_2012Metric_Pad1.18x1.45mm_HandSolder, F.Cu at (183.8, -37.9)
- added C76: 0.1uF, Capacitor_SMD:C_0805_2012Metric_Pad1.18x1.45mm_HandSolder, F.Cu at (204.5, -67.8)
- added C77: 0.1uF, Capacitor_SMD:C_0805_2012Metric_Pad1.18x1.45mm_HandSolder, F.Cu at (204.5, -64.8)
- added R10: 10K, Resistor_SMD:R_0805_2012Metric_Pad1.20x1.40mm_HandSolder, F.Cu at (188.6, -41.3)
- added R11: 10K, Resistor_SMD:R_0805_2012Metric_Pad1.20x1.40mm_HandSolder, F.Cu at (188.6, -38.3)
- added R6: 22R, Resistor_SMD:R_0805_2012Metric_Pad1.20x1.40mm_HandSolder, F.Cu at (188.6, -53.1)
- added R7: 22R, Resistor_SMD:R_0805_2012Metric_Pad1.20x1.40mm_HandSolder, F.Cu at (188.6, -50.1)
- added R8: 4K7, Resistor_SMD:R_0805_2012Metric_Pad1.20x1.40mm_HandSolder, F.Cu at (188.6, -47.2)
- added R9: 1K, Resistor_SMD:R_0805_2012Metric_Pad1.20x1.40mm_HandSolder, F.Cu at (188.6, -44.2)
- added RN3: 4K7, Resistor_THT:R_Array_SIP5, F.Cu at (111.9, 135.2)
- added RN4: 22R, Package_SO:SOIC-16W_5.3x10.2mm_P1.27mm, F.Cu at (167.4, -63.4)
- added RN5: 22R, Package_SO:SOIC-16W_5.3x10.2mm_P1.27mm, F.Cu at (177.8, -63.4)
- added RN6: 22R, Package_SO:SOIC-16W_5.3x10.2mm_P1.27mm, F.Cu at (188.3, -63.4)
- added TP1: TP_VCLK, TestPoint:TestPoint_Loop_D1.80mm_Drill1.0mm_Beaded, F.Cu at (188.5, -34.5)
- added TP2: TP_DA0, TestPoint:TestPoint_Loop_D1.80mm_Drill1.0mm_Beaded, F.Cu at (188.5, -29.9)
- added TP3: TP_OSC, TestPoint:TestPoint_Loop_D1.80mm_Drill1.0mm_Beaded, F.Cu at (188.5, -25.2)
- added U16: MAX3012, Package_SO:TSSOP-20_4.4x6.5mm_P0.65mm, F.Cu at (195.7, -53.5)
- added U18: XC6SLX9-2TQG144I, Dragon:AMD-LQFP-144, F.Cu at (259.4, 137.1)
- added U19: SN105125DBVR, Package_TO_SOT_SMD:SOT-23-5, F.Cu at (193.4, -34.4)
- added U20: SN105125DBVR, Package_TO_SOT_SMD:SOT-23-5, F.Cu at (193.4, -29.8)
- added U21: MAX3012, Package_SO:TSSOP-20_4.4x6.5mm_P0.65mm, F.Cu at (195.7, -45.4)
- added X3: 14.31818MHz, Oscillator:Oscillator_SMD_ECS_2520MV-xxx-xx-4Pin_2.5x2.0mm, F.Cu at (197.9, -34.7)
- C17: value 100n -> 100uF; footprint Capacitor_SMD:C_0805_2012Metric_Pad1.18x1.45mm_HandSolder -> Capacitor_SMD:C_0805_2012Metric
- C18, C19: value 1u -> 0.1uF; footprint Capacitor_Tantalum_SMD:CP_EIA-3216-18_Kemet-A_Pad1.58x1.35mm_HandSolder -> Capacitor_SMD:C_0805_2012Metric_Pad1.18x1.45mm_HandSolder
- C2: value 10uF -> 10u
- C6: value 4.7uF -> 0.1uF; footprint Capacitor_Tantalum_SMD:CP_EIA-3216-18_Kemet-A_Pad1.58x1.35mm_HandSolder -> Capacitor_SMD:C_0805_2012Metric_Pad1.18x1.45mm_HandSolder
- D10: value 1N914 -> LED_RED; footprint Diode_SMD:D_SOD-323_HandSoldering -> LED_SMD:LED_0805_2012Metric
- JP1: value 32k/64k -> Enable 8M; footprint Connector_PinHeader_2.54mm:PinHeader_1x03_P2.54mm_Vertical -> Jumper:SolderJumper-2_P1.3mm_Open_Pad1.0x1.5mm
- PL7: footprint Dragon:Edge_2x20_P2.54mm_OvalMP -> Connector_PinHeader_2.54mm:PinHeader_2x20_P2.54mm_Vertical
- PL8: footprint Connector_PinHeader_2.54mm:PinHeader_2x20_P2.54mm_Vertical -> Dragon:Edge_2x20_P2.54mm_OvalMP
- R3: value 22R -> 100R; moved to F.Cu
- U1: value AS6C1008-TIN -> MAX3012; footprint Package_SO:TSOP-I-32_18.4x8mm_P0.5mm -> Package_SO:TSSOP-20_4.4x6.5mm_P0.65mm
- U12: value 6551 -> W65C51; footprint Package_DIP:DIP-28_W15.24mm -> Package_LCC:PLCC-28_SMD-Socket
- U13: value 4069 -> RMLV3216A; footprint Package_SO:SOIC-14_3.9x8.7mm_P1.27mm -> Package_SO:TSOP-I-48_18.4x12mm_P0.5mm
- U14: value LM348DR -> 74AHCT1G04; footprint Package_SO:SOIC-14_3.9x8.7mm_P1.27mm -> Package_TO_SOT_SMD:SOT-23-5_HandSoldering
- U2: value AS6C1008-55TIN -> MAX3012; footprint Package_SO:TSOP-I-32_18.4x8mm_P0.5mm -> Package_SO:TSSOP-20_4.4x6.5mm_P0.65mm
- U3: value XC95144XL-TQ100 -> SST39SF040-55; footprint Package_QFP:TQFP-100_14x14mm_P0.5mm -> Package_LCC:PLCC-32_THT-Socket
- U7: value W65C21 -> MAX232; footprint Package_LCC:PLCC-44_SMD-Socket -> Package_SO:SOIC-16_3.9x9.9mm_P1.27mm
- U8: value 28C256 -> 74HCT244; footprint Package_LCC:PLCC-32_THT-Socket -> Package_SO:TSSOP-20_4.4x6.5mm_P0.65mm
- U9: value 74HCT1G08 -> 74HCT244; footprint Package_TO_SOT_SMD:SOT-353_SC-70-5_Handsoldering -> Package_SO:TSSOP-20_4.4x6.5mm_P0.65mm
- moved U13 134.6 mm to (261.6, 61.0)
- moved C17 125.7 mm to (193.1, -26.1), turned to 0 degrees
- moved R3 121.6 mm to (188.6, -56.0), turned to 0 degrees
- moved C22 121.1 mm to (111.3, 115.4)
- moved IC19 120.6 mm to (117.8, 108.7)
- moved D10 119.3 mm to (197.5, -26.1)
- moved C18 97.0 mm to (164.5, -56.0), turned to 0 degrees
- moved C19 92.1 mm to (164.5, -53.0), turned to 0 degrees
- moved U7 68.1 mm to (122.0, 64.8), turned to 180 degrees
- moved C2 60.0 mm to (126.0, 75.4), turned to 90 degrees
- moved C10 29.5 mm to (127.6, 68.1)
- moved R15 26.2 mm to (257.1, 165.4)
- moved U14 26.0 mm to (151.5, 67.8)
- moved U9 21.8 mm to (203.3, 137.2)
- moved IC10 21.8 mm to (185.5, 138.2)
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Connections:
- C1 pad 1: GND -> SLOT2SZ0
- C10 pad 2: GND -> SLOT2SZ0
- C11 pad 2: GND -> SLOT2SZ0
- C12 pad 2: GND -> SLOT2SZ0
- C13 pad 2: GND -> SLOT2SZ0
- C14 pad 2: GND -> SLOT2SZ0
- C15 pad 2: GND -> SLOT2SZ0
- C16 pad 2: GND -> SLOT2SZ0
- C17 pad 1: +12V -> SLOT2SZ0
- C17 pad 2: GND -> +3V3
- C18 pad 1: GND -> SLOT2SZ0
- C18 pad 2: -5V -> +3V3
- C19 pad 1: GND -> SLOT2SZ0
- C19 pad 2: -12V -> +3V3
- C2 pad 1: +5V -> Net-(U7-C1+)
- C2 pad 2: GND -> Net-(U7-C1-)
- C22 pad 2: GND -> SLOT2SZ0
- C23 pad 2: GND -> SLOT2SZ0
- C26 pad 1: GND -> SLOT2SZ0
- C3 pad 1: GND -> SLOT2SZ0
- C3 pad 2: +5V -> +3V3
- C30 pad 1: GND -> SLOT2SZ0
- C31 pad 1: GND -> SLOT2SZ0
- C32 pad 1: GND -> SLOT2SZ0
- C33 pad 1: GND -> SLOT2SZ0
- C38 pad 1: GND -> SLOT2SZ0
- C39 pad 1: GND -> SLOT2SZ0
- C4 pad 2: GND -> SLOT2SZ0
- C42 pad 2: GND -> SLOT2SZ0
- C43 pad 2: GND -> SLOT2SZ0
- C44 pad 1: GND -> SLOT2SZ0
- C45 pad 2: GND -> SLOT2SZ0
- C48 pad 1: GND -> SLOT2SZ0
- C5 pad 1: GND -> +5V
- C5 pad 2: +5V -> SLOT2SZ0
- C6 pad 2: GND -> SLOT2SZ0
- C68 pad 1: GND -> SLOT2SZ0
- C69 pad 1: GND -> SLOT2SZ0
- C7 pad 2: GND -> SLOT2SZ0
- C8 pad 2: GND -> SLOT2SZ0
- C9 pad 2: GND -> SLOT2SZ0
- D10 pad 2: Net-(D10-A) -> +3V3
- D7 pad 2: GND -> SLOT2SZ0
- D9 pad 2: GND -> SLOT2SZ0
- IC1 pad 4: GND -> SLOT2SZ0
- IC10 pad 8: GND -> SLOT2SZ0
- IC19 pad 1: GND -> SLOT2SZ0
- IC19 pad 13: A5 -> /MPU/A5
- IC19 pad 14: A6 -> /MPU/A6
- IC19 pad 15: A7 -> /MPU/A7
- IC19 pad 16: A8 -> /MPU/A8
- IC19 pad 17: A9 -> /MPU/A9
- IC19 pad 18: A10 -> /MPU/A10
- IC19 pad 19: A11 -> /MPU/A11
- IC19 pad 20: A12 -> /MPU/A12
- IC19 pad 21: A13 -> /MPU/A13
- IC19 pad 22: A14 -> /MPU/A14
- IC19 pad 23: A15 -> /MPU/A15
- IC19 pad 24: D7 -> /AUDIO/DC7
- IC19 pad 25: D6 -> /AUDIO/DC6
- IC19 pad 26: D5 -> /AUDIO/DC5
- IC19 pad 27: D4 -> /AUDIO/DC4
- IC19 pad 28: D3 -> /AUDIO/DC3
- IC19 pad 29: D2 -> /AUDIO/DC2
- IC19 pad 30: D1 -> /AUDIO/DC1
- IC19 pad 31: D0 -> /AUDIO/DC0
- IC19 pad 33: GND -> SLOT2SZ0
- IC19 pad 36: GND -> SLOT2SZ0
- IC19 pad 38: GND -> SLOT2SZ0
- IC19 pad 39: GND -> SLOT2SZ0
- IC19 pad 5: GND -> SLOT2SZ0
- IC19 pad 6: GND -> SLOT2SZ0
- IC19 pad 8: A0 -> /MPU/A0
- IC19 pad 9: A1 -> /MPU/A1
- IC24 pad 1: GND -> SLOT2SZ0
- IC24 pad 10: GND -> SLOT2SZ0
- IC24 pad 19: GND -> SLOT2SZ0
- IC31 pad 1: Net-(JP1-B) -> Net-(IC33-E2)
- IC31 pad 7: GND -> SLOT2SZ0
- IC33 pad 8: GND -> SLOT2SZ0
- IC34 pad 8: GND -> SLOT2SZ0
- J1 pad 5: GND -> SLOT2SZ0
- J2 pad 11: DO4 -> /MPU/D4
- J2 pad 13: DO5 -> /MPU/D5
- J2 pad 15: DO6 -> /MPU/D6
- J2 pad 17: DO7 -> /MPU/D7
- J2 pad 3: DO0 -> /MPU/D0
- J2 pad 4: GND -> SLOT2SZ0
- J2 pad 5: DO1 -> /MPU/D1
- J2 pad 7: DO2 -> /MPU/D2
- J2 pad 9: DO3 -> /MPU/D3
- J3 pad 1: DC0 -> unconnected-(J3-Pin_1-Pad1)
- J3 pad 10: RC -> unconnected-(J3-Pin_10-Pad10)
- J3 pad 11: DC5 -> unconnected-(J3-Pin_11-Pad11)
- J3 pad 12: unconnected-(J3-Pin_12-Pad12) -> P1b
- J3 pad 13: DC6 -> unconnected-(J3-Pin_13-Pad13)
- J3 pad 14: unconnected-(J3-Pin_14-Pad14) -> R/~{W}
- J3 pad 15: DC7 -> unconnected-(J3-Pin_15-Pad15)
- J3 pad 16: unconnected-(J3-Pin_16-Pad16) -> E
- J3 pad 2: Alpha -> unconnected-(J3-Pin_2-Pad2)
- J3 pad 3: DC1 -> unconnected-(J3-Pin_3-Pad3)
- J3 pad 4: Inverse -> unconnected-(J3-Pin_4-Pad4)
- J3 pad 5: DC2 -> unconnected-(J3-Pin_5-Pad5)
- J3 pad 6: ~{SelInv} -> unconnected-(J3-Pin_6-Pad6)
- J3 pad 7: DC3 -> unconnected-(J3-Pin_7-Pad7)
- J3 pad 8: RClk -> unconnected-(J3-Pin_8-Pad8)
- J3 pad 9: DC4 -> unconnected-(J3-Pin_9-Pad9)
- J4 pad 2: GND -> SLOT2SZ0
- J6 pad 10: D1 -> /AUDIO/DC1
- J6 pad 11: D0 -> /AUDIO/DC0
- J6 pad 12: D7 -> /AUDIO/DC7
- J6 pad 13: D6 -> /AUDIO/DC6
- J6 pad 17: GND -> SLOT2SZ0
- J6 pad 2: GND -> SLOT2SZ0
- J6 pad 20: GND -> SLOT2SZ0
- J6 pad 6: D5 -> /AUDIO/DC5
- J6 pad 7: D4 -> /AUDIO/DC4
- J6 pad 8: D2 -> /AUDIO/DC2
- J6 pad 9: D3 -> /AUDIO/DC3
- J7 pad 10: D1 -> /AUDIO/DC1
- J7 pad 11: D0 -> /AUDIO/DC0
- J7 pad 12: D7 -> /AUDIO/DC7
- J7 pad 13: D6 -> /AUDIO/DC6
- J7 pad 17: GND -> SLOT2SZ0
- J7 pad 2: GND -> SLOT2SZ0
- J7 pad 20: GND -> SLOT2SZ0
- J7 pad 6: D5 -> /AUDIO/DC5
- J7 pad 7: D4 -> /AUDIO/DC4
- J7 pad 8: D2 -> /AUDIO/DC2
- J7 pad 9: D3 -> /AUDIO/DC3
- J8 pad 2: GND -> SLOT2SZ0
- JP1 pad 1: GND -> Z22
- JP1 pad 2: Net-(IC33-E2) -> Net-(JP1-B)
- JP4 pad 2: GND -> SLOT2SZ0
- PL1 pad 5: GND -> SLOT2SZ0
- PL2 pad 10: GND -> SLOT2SZ0
- PL2 pad 12: GND -> SLOT2SZ0
- PL2 pad 14: GND -> SLOT2SZ0
- PL2 pad 16: GND -> SLOT2SZ0
- PL2 pad 18: GND -> SLOT2SZ0
- PL2 pad 6: GND -> SLOT2SZ0
- PL2 pad 8: GND -> SLOT2SZ0
- PL3 pad 3: GND -> SLOT2SZ0
- PL4 pad 2: GND -> SLOT2SZ0
- PL5 pad 3: GND -> SLOT2SZ0
- PL6 pad 5: GND -> SLOT2SZ0
- PL6 pad 6: GND -> SLOT2SZ0
- PL6 pad 7: -12V -> -5V
- PL7 pad 10: D0 -> /AUDIO/DC0
- PL7 pad 11: D1 -> /AUDIO/DC1
- PL7 pad 12: D2 -> /AUDIO/DC2
- PL7 pad 13: D3 -> /AUDIO/DC3
- PL7 pad 14: D4 -> /AUDIO/DC4
- PL7 pad 15: D5 -> /AUDIO/DC5
- PL7 pad 16: D6 -> /AUDIO/DC6
- PL7 pad 17: D7 -> /AUDIO/DC7
- PL7 pad 19: A0 -> /CARTRIDGE/CA0
- PL7 pad 20: A1 -> /CARTRIDGE/CA1
- PL7 pad 21: A2 -> /CARTRIDGE/CA2
- PL7 pad 22: A3 -> /CARTRIDGE/CA3
- PL7 pad 23: A4 -> /CARTRIDGE/CA4
- PL7 pad 24: A5 -> /CARTRIDGE/CA5
- PL7 pad 25: A6 -> /CARTRIDGE/CA6
- PL7 pad 26: A7 -> /CARTRIDGE/CA7
- PL7 pad 27: A8 -> /CARTRIDGE/CA8
- PL7 pad 28: A9 -> /CARTRIDGE/CA9
- PL7 pad 29: A10 -> /CARTRIDGE/CA10
- PL7 pad 30: A11 -> /CARTRIDGE/CA11
- PL7 pad 31: A12 -> /CARTRIDGE/CA12
- PL7 pad 33: GND -> SLOT2SZ0
- PL7 pad 34: GND -> SLOT2SZ0
- PL7 pad 37: A13 -> /CARTRIDGE/CA13
- PL7 pad 38: A14 -> /CARTRIDGE/CA14
- PL7 pad 39: A15 -> /CARTRIDGE/CA15
- PL8 pad 10: D0 -> /AUDIO/DC0
- PL8 pad 11: D1 -> /AUDIO/DC1
- PL8 pad 12: D2 -> /AUDIO/DC2
- PL8 pad 13: D3 -> /AUDIO/DC3
- PL8 pad 14: D4 -> /AUDIO/DC4
- PL8 pad 15: D5 -> /AUDIO/DC5
- PL8 pad 16: D6 -> /AUDIO/DC6
- PL8 pad 17: D7 -> /AUDIO/DC7
- PL8 pad 19: A0 -> /CARTRIDGE/CA0
- PL8 pad 20: A1 -> /CARTRIDGE/CA1
- PL8 pad 21: A2 -> /CARTRIDGE/CA2
- PL8 pad 22: A3 -> /CARTRIDGE/CA3
- PL8 pad 23: A4 -> /CARTRIDGE/CA4
- PL8 pad 24: A5 -> /CARTRIDGE/CA5
- PL8 pad 25: A6 -> /CARTRIDGE/CA6
- PL8 pad 26: A7 -> /CARTRIDGE/CA7
- PL8 pad 27: A8 -> /CARTRIDGE/CA8
- PL8 pad 28: A9 -> /CARTRIDGE/CA9
- PL8 pad 29: A10 -> /CARTRIDGE/CA10
- PL8 pad 30: A11 -> /CARTRIDGE/CA11
- PL8 pad 31: A12 -> /CARTRIDGE/CA12
- PL8 pad 33: GND -> SLOT2SZ0
- PL8 pad 34: GND -> SLOT2SZ0
- PL8 pad 37: A13 -> /CARTRIDGE/CA13
- PL8 pad 38: A14 -> /CARTRIDGE/CA14
- PL8 pad 39: A15 -> /CARTRIDGE/CA15
- PL9 pad 1: GND -> SLOT2SZ0
- PL9 pad 2: Net-(PL9-Pad2) -> /Serial/x~{CTS}
- PL9 pad 4: Net-(PL9-Pad4) -> /Serial/x~{DTR}
- PL9 pad 5: Net-(PL9-Pad5) -> /Serial/xRxD
- PL9 pad 6: Net-(PL9-Pad6) -> /Serial/xTxD
- R16 pad 1: GND -> SLOT2SZ0
- R3 pad 1: ~{CAS} -> VCLK
- R3 pad 2: Net-(U3-P68) -> Net-(U18D-IO_L1P_3)
- R30 pad 1: GND -> SLOT2SZ0
- R46 pad 1: GND -> SLOT2SZ0
- R48 pad 1: GND -> SLOT2SZ0
- R53 pad 2: -12V -> -5V
- R68 pad 1: GND -> SLOT2SZ0
- R75 pad 1: GND -> SLOT2SZ0
- SW1 pad 2: unconnected-(SW1-B-Pad2) -> SLOT2SZ0
- SW1 pad 5: GND -> SLOT2SZ0
- TR1 pad 3: GND -> SLOT2SZ0
- U1 pad 1: Z11 -> /MPU/D7
- U1 pad 10: Z16 -> ~{CPU_WRITE}
- U1 pad 11: Z14 -> SLOT2SZ0
- U1 pad 12: Z12 -> /AUDIO/DC0
- U1 pad 13: Z7 -> /AUDIO/DC1
- U1 pad 14: Z6 -> /AUDIO/DC2
- U1 pad 15: Z5 -> /AUDIO/DC3
- U1 pad 16: Z4 -> /AUDIO/DC4
- U1 pad 17: Z3 -> /AUDIO/DC5
- U1 pad 18: Z2 -> /AUDIO/DC6
- U1 pad 19: Z1 -> +5V
- U1 pad 2: Z9 -> +3V3
- U1 pad 20: Z0 -> /AUDIO/DC7
- U1 pad 3: Z8 -> /MPU/D6
- U1 pad 4: Z13 -> /MPU/D5
- U1 pad 5: R/~{W} -> /MPU/D4
- U1 pad 6: +5V -> /MPU/D3
- U1 pad 7: Z15 -> /MPU/D2
- U1 pad 8: +5V -> /MPU/D1
- U1 pad 9: unconnected-(U1-NC-Pad9) -> /MPU/D0
- U10 pad 4: GND -> SLOT2SZ0
- U10 pad 6: GND -> SLOT2SZ0
- U10 pad 7: GND -> SLOT2SZ0
- U10 pad 8: GND -> SLOT2SZ0
- U11 pad 3: GND -> SLOT2SZ0
- U12 pad 1: GND -> SLOT2SZ0
- U12 pad 10: Net-(U12-TXD) -> /Serial/TxD
- U12 pad 11: Net-(U12-~{DTR}) -> /Serial/~{DTR}
- U12 pad 12: Net-(U12-RXD) -> /Serial/RxD
- U12 pad 13: A0 -> Z0
- U12 pad 14: A1 -> Z1
- U12 pad 16: GND -> SLOT2SZ0
- U12 pad 17: GND -> SLOT2SZ0
- U12 pad 18: D0 -> /AUDIO/DC0
- U12 pad 19: D1 -> /AUDIO/DC1
- U12 pad 2: A2 -> Z2
- U12 pad 20: D2 -> /AUDIO/DC2
- U12 pad 21: D3 -> /AUDIO/DC3
- U12 pad 22: D4 -> /AUDIO/DC4
- U12 pad 23: D5 -> /AUDIO/DC5
- U12 pad 24: D6 -> /AUDIO/DC6
- U12 pad 25: D7 -> /AUDIO/DC7
- U12 pad 9: Net-(U12-~{CTS}) -> /Serial/~{CTS}
- U13 pad 1: Net-(D14-A) -> Z20
- U13 pad 10: Net-(U14C-IN+) -> Z11
- U13 pad 11: Net-(U12-~{DTR}) -> R/~{W}
- U13 pad 12: Net-(U12-RXD) -> +3V3
- U13 pad 13: Net-(D16-A) -> Net-(JP1-B)
- U13 pad 14: +5V -> unconnected-(U13-~{UB}-Pad14)
- U13 pad 2: Net-(U12-~{CTS}) -> Z19
- U13 pad 3: unconnected-(U13-Pad3) -> Z18
- U13 pad 4: unconnected-(U13-Pad4) -> Z17
- U13 pad 5: Net-(U12-TXD) -> Z16
- U13 pad 6: Net-(U14B-IN-) -> Z15
- U13 pad 7: GND -> Z14
- U13 pad 8: Net-(JP3-A) -> Z13
- U13 pad 9: A2 -> Z12
- U14 pad 1: Net-(U14A-OUT) -> (no net)
- U14 pad 2: Net-(D12-A) -> A2
- U14 pad 3: Net-(D12-K) -> SLOT2SZ0
- U14 pad 4: +12V -> Net-(JP3-A)
- U14 pad 5: Net-(U12-TXD) -> +5V
- U17 pad 10: A1 -> Z1
- U17 pad 13: A1 -> Z1
- U17 pad 2: A0 -> Z0
- U17 pad 5: A0 -> Z0
- U17 pad 7: GND -> SLOT2SZ0
- U2 pad 1: Z11 -> /SAM/zA8
- U2 pad 10: Z16 -> +3V3
- U2 pad 11: Z14 -> SLOT2SZ0
- U2 pad 12: Z12 -> /MPU/A15
- U2 pad 13: Z7 -> /MPU/A14
- U2 pad 14: Z6 -> /MPU/A13
- U2 pad 15: Z5 -> /MPU/A12
- U2 pad 16: Z4 -> /MPU/A11
- U2 pad 17: Z3 -> /MPU/A10
- U2 pad 18: Z2 -> /MPU/A9
- U2 pad 19: Z1 -> +5V
- U2 pad 2: Z9 -> +3V3
- U2 pad 20: Z0 -> /MPU/A8
- U2 pad 3: Z8 -> /SAM/zA9
- U2 pad 4: Z13 -> /SAM/zA10
- U2 pad 5: R/~{W} -> /SAM/zA11
- U2 pad 6: Z17 -> /SAM/zA12
- U2 pad 7: Z15 -> /SAM/zA13
- U2 pad 8: +5V -> /SAM/zA14
- U2 pad 9: unconnected-(U2-NC-Pad9) -> /SAM/zA15
- U3 pad 1: Net-(U3-I/O/GTS3) -> Z18
- U3 pad 10: GND -> Z2
- U3 pad 11: GND -> Z1
- U3 pad 12: A12 -> Z0
- U3 pad 13: GND -> /MPU/D0
- U3 pad 14: A13 -> /MPU/D1
- U3 pad 15: GND -> /MPU/D2
- U3 pad 16: GND -> SLOT2SZ0
- U3 pad 17: A8 -> /MPU/D3
- U3 pad 18: A9 -> /MPU/D4
- U3 pad 19: A10 -> /MPU/D5
- U3 pad 2: GND -> Z16
- U3 pad 20: A11 -> /MPU/D6
- U3 pad 21: GND -> /MPU/D7
- U3 pad 22: DA0 -> SLOT2SZ0
- U3 pad 23: /SAM/OSC -> Z10
- U3 pad 24: GND -> ~{ROM}
- U3 pad 25: GND -> Z11
- U3 pad 26: +3V3 -> Z9
- U3 pad 27: GND -> Z8
- U3 pad 28: GND -> Z13
- U3 pad 29: GND -> Z14
- U3 pad 3: GND -> Z15
- U3 pad 30: GND -> Z17
- U3 pad 31: GND -> ~{ROM2}
- U3 pad 32: GND -> +5V
- U3 pad 4: GND -> Z12
- U3 pad 5: +3V3 -> Z7
- U3 pad 6: GND -> Z6
- U3 pad 7: GND -> Z5
- U3 pad 8: A15 -> Z4
- U3 pad 9: A14 -> Z3
- U4 pad 2: GND -> SLOT2SZ0
- U5 pad 1: GND -> SLOT2SZ0
- U5 pad 29: D7 -> /AUDIO/DC7
- U5 pad 30: D6 -> /AUDIO/DC6
- U5 pad 31: D5 -> /AUDIO/DC5
- U5 pad 32: D4 -> /AUDIO/DC4
- U5 pad 33: D3 -> /AUDIO/DC3
- U5 pad 34: D2 -> /AUDIO/DC2
- U5 pad 35: D1 -> /AUDIO/DC1
- U5 pad 36: D0 -> /AUDIO/DC0
- U6 pad 1: GND -> SLOT2SZ0
- U6 pad 29: D7 -> /AUDIO/DC7
- U6 pad 30: D6 -> /AUDIO/DC6
- U6 pad 31: D5 -> /AUDIO/DC5
- U6 pad 32: D4 -> /AUDIO/DC4
- U6 pad 33: D3 -> /AUDIO/DC3
- U6 pad 34: D2 -> /AUDIO/DC2
- U6 pad 35: D1 -> /AUDIO/DC1
- U6 pad 36: D0 -> /AUDIO/DC0
- U7 pad 1: GND -> Net-(U7-C1+)
- U7 pad 10: DC7 -> /Serial/~{DTR}
- U7 pad 11: RC -> /Serial/TxD
- U7 pad 12: RClk -> /Serial/RxD
- U7 pad 13: ~{SelInv} -> /Serial/xRxD
- U7 pad 14: Inverse -> /Serial/xTxD
- U7 pad 15: Alpha -> SLOT2SZ0
- U7 pad 16: unconnected-(U7-PB5-Pad16) -> +5V
- U7 pad 2: unconnected-(U7-NC-Pad2) -> Net-(U7-VS+)
- U7 pad 3: DC0 -> Net-(U7-C1-)
- U7 pad 4: DC1 -> Net-(U7-C2+)
- U7 pad 5: DC2 -> Net-(U7-C2-)
- U7 pad 6: DC3 -> Net-(U7-VS-)
- U7 pad 7: DC4 -> /Serial/x~{DTR}
- U7 pad 8: DC5 -> /Serial/x~{CTS}
- U7 pad 9: DC6 -> /Serial/~{CTS}
- U8 pad 1: unconnected-(U8-DC-Pad1) -> E
- U8 pad 10: A1 -> SLOT2SZ0
- U8 pad 11: A0 -> Z4
- U8 pad 12: unconnected-(U8-NC-Pad12) -> /CARTRIDGE/CA3
- U8 pad 13: D0 -> Z5
- U8 pad 14: D1 -> /CARTRIDGE/CA2
- U8 pad 15: D2 -> Z6
- U8 pad 16: GND -> /CARTRIDGE/CA1
- U8 pad 17: unconnected-(U8-DC-Pad17) -> Z7
- U8 pad 18: D3 -> /CARTRIDGE/CA0
- U8 pad 19: D4 -> SLOT2SZ0
- U8 pad 2: Net-(JP6-Out) -> Z0
- U8 pad 20: D5 -> +5V
- U8 pad 3: A12 -> /CARTRIDGE/CA7
- U8 pad 4: A7 -> Z1
- U8 pad 5: A6 -> /CARTRIDGE/CA6
- U8 pad 6: A5 -> Z2
- U8 pad 7: A4 -> /CARTRIDGE/CA5
- U8 pad 8: A3 -> Z3
- U8 pad 9: A2 -> /CARTRIDGE/CA4
- U9 pad 1: ~{E18} -> E
- U9 pad 2: ~{E17} -> Z8
- U9 pad 3: GND -> /CARTRIDGE/CA15
- U9 pad 4: ~{ROM} -> Z9
- U9 pad 5: +5V -> /CARTRIDGE/CA14
- X2 pad 3: GND -> SLOT2SZ0
Routing:
- net +5V: track 1640.1 -> 0.00 mm, vias 38 -> 0
- net R/~{W}: track 610.0 -> 0.00 mm, vias 16 -> 0
- net A0: track 594.2 -> 0.00 mm, vias 13 -> 0
- net A1: track 580.7 -> 0.00 mm, vias 13 -> 0
- net ~{RES}: track 578.7 -> 0.00 mm, vias 9 -> 0
- net D7: track 574.5 -> 0.00 mm, vias 13 -> 0
- net D6: track 570.7 -> 0.00 mm, vias 12 -> 0
- net D4: track 558.8 -> 0.00 mm, vias 13 -> 0
- net D5: track 558.0 -> 0.00 mm, vias 12 -> 0
- net D1: track 551.3 -> 0.00 mm, vias 12 -> 0
- net D0: track 543.5 -> 0.00 mm, vias 12 -> 0
- net D3: track 535.8 -> 0.00 mm, vias 11 -> 0
- net D2: track 534.0 -> 0.00 mm, vias 13 -> 0
- net E: track 532.4 -> 0.00 mm, vias 13 -> 0
- net +12V: track 450.8 -> 0.00 mm, vias 4 -> 0
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- added copper zone on B.Cu, net SLOT2SZ0
- added copper zone on F.Cu, net SLOT2SZ0
- removed copper zone on B.Cu, net GND
- removed copper zone on F.Cu, net GND
Other:
- board text added: "Riven"
- board text added: "SIDE 1"
- board text removed: "locked"

Commit message: rework traces for FPGA
Parts:
- removed C70: 4.7uF, Capacitor_SMD:C_0805_2012Metric_Pad1.18x1.45mm_HandSolder
- removed C71, C72, C73: 0.47uF, Capacitor_SMD:C_0805_2012Metric_Pad1.18x1.45mm_HandSolder
- removed C74, C75: 0.1uF, Capacitor_SMD:C_0805_2012Metric_Pad1.18x1.45mm_HandSolder
- removed IC10: 74ACT138, Package_SO:SOIC-16W_7.5x10.3mm_P1.27mm
- removed IC33: 74ACT138N, Package_SO:SOIC-16W_7.5x10.3mm_P1.27mm
- removed R39: 4K7, Resistor_SMD:R_0805_2012Metric_Pad1.20x1.40mm_HandSolder
- added IC2: 74ACT02, Package_SO:SOIC-14_3.9x8.7mm_P1.27mm, F.Cu at (229.6, 185.1)
- added IC3: 74ACT138N, Package_SO:SOIC-16W_7.5x10.3mm_P1.27mm, F.Cu at (241.6, 185.8)
- added IC4: 74ACT138, Package_SO:SOIC-16W_7.5x10.3mm_P1.27mm, F.Cu at (114.8, 110.4)
- added JP6: SZ1, Jumper:SolderJumper-2_P1.3mm_Open_Pad1.0x1.5mm, B.Cu at (262.2, 142.9)
- added JP7: SZ2, Jumper:SolderJumper-2_P1.3mm_Bridged_Pad1.0x1.5mm, B.Cu at (262.2, 140.4)
- added R12: 4K7, Resistor_SMD:R_0805_2012Metric_Pad1.20x1.40mm_HandSolder, B.Cu at (258.7, 145.4)
- added R13: 4K7, Resistor_SMD:R_0805_2012Metric_Pad1.20x1.40mm_HandSolder, B.Cu at (258.7, 142.9)
- added R14: 4K7, Resistor_SMD:R_0805_2012Metric_Pad1.20x1.40mm_HandSolder, B.Cu at (258.7, 140.3)
- added R2: 4K7, Resistor_SMD:R_0805_2012Metric_Pad1.20x1.40mm_HandSolder, F.Cu at (292.0, 160.4)
- added R4: 22R, Resistor_SMD:R_0805_2012Metric_Pad1.20x1.40mm_HandSolder, B.Cu at (292.1, 156.5)
- added R5: 22R, Resistor_SMD:R_0805_2012Metric_Pad1.20x1.40mm_HandSolder, F.Cu at (292.0, 158.4)
- added U15: 74LS373, Package_SO:SOIC-20W_7.5x12.8mm_P1.27mm, F.Cu at (263.1, 76.8)
- C1, C10, C40, C41, C44, C49, C54, C57, C61, C62, C76, C77, R45, R46, R47, R52: moved to B.Cu
- C11, C7: value 100n -> 0.1uF
- C12, C13, C14, C15, C16: value 100n -> 4.7uF
- C17: value 100uF -> 4.7uF; footprint Capacitor_SMD:C_0805_2012Metric -> Capacitor_SMD:C_0805_2012Metric_Pad1.18x1.45mm_HandSolder; moved to B.Cu
- C18, C19, C28: value 0.1uF -> 4.7uF; moved to B.Cu
- C25: value 0.1uF -> 0.47uF; moved to B.Cu
- C29, C34, C52, C56, C59: value 4.7uF -> 0.47uF; moved to B.Cu
- C36: value 0.47uF -> 0.1uF; moved to B.Cu
- C37, C50: value 0.47uF -> 4.7uF; moved to B.Cu
- C47: value 4.7uF -> 0.1uF; moved to B.Cu
- C53: value 4.7uF -> 100uF; moved to B.Cu
- C55: value 1u -> 4.7uF; moved to B.Cu
- C58: value 1u -> 0.47uF; moved to B.Cu
- C60: value 0.47uF -> 0.01uF; moved to B.Cu
- C63: value 0.01uF -> 1u; moved to B.Cu
- C64: value 4.7uF -> 2u2; moved to B.Cu
- C65: value 4.7uF -> 100n; moved to B.Cu
- C66, C67: value 4.7uF -> 1u; moved to B.Cu
- C8: value 1u -> 0.1uF
- C9: value 2u2 -> 0.1uF
- JP1: value Enable 8M -> SZ0; footprint Jumper:SolderJumper-2_P1.3mm_Open_Pad1.0x1.5mm -> Jumper:SolderJumper-2_P1.3mm_Bridged_Pad1.0x1.5mm; moved to B.Cu
- R6: value 22R -> 4K7
- R7: value 22R -> 4K7; moved to B.Cu
- R8: value 4K7 -> 1K
- R9: value 1K -> 4K7; moved to B.Cu
- U9: moved to F.Cu
- moved C60 248.9 mm to (275.6, 173.4)
- moved C37 248.8 mm to (285.8, 163.9), turned to 180 degrees
- moved U16 246.4 mm to (281.9, 177.4), turned to -90 degrees
- moved C63 245.7 mm to (288.6, 173.0), turned to -90 degrees
- moved RN5 245.1 mm to (252.7, 170.0), turned to 180 degrees
- moved C64 243.9 mm to (290.6, 173.0), turned to -90 degrees
- moved C25 242.4 mm to (285.8, 159.9)
- moved C41 241.8 mm to (285.8, 161.9), turned to 180 degrees
- moved C34 241.1 mm to (285.8, 167.4), turned to 180 degrees
- moved C55 239.9 mm to (274.5, 167.9), turned to 90 degrees
- moved C18 239.7 mm to (283.1, 152.3), turned to -90 degrees
- moved C49 239.3 mm to (280.5, 167.9), turned to 90 degrees
- moved C65 239.0 mm to (261.3, 183.4), turned to 180 degrees
- moved R6 239.0 mm to (292.1, 162.3)
- moved C54 238.7 mm to (285.8, 158.0), turned to 180 degrees
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Connections:
- net ~{CPU_WRITE} renamed CPU_WRITE
- C1 pad 1: SLOT2SZ0 -> GND
- C10 pad 2: SLOT2SZ0 -> GND
- C11 pad 1: +3V3 -> +5V
- C11 pad 2: SLOT2SZ0 -> GND
- C12 pad 1: +3V3 -> +1V2
- C12 pad 2: SLOT2SZ0 -> GND
- C13 pad 2: SLOT2SZ0 -> GND
- C14 pad 1: +3V3 -> +1V2
- C14 pad 2: SLOT2SZ0 -> GND
- C15 pad 2: SLOT2SZ0 -> GND
- C16 pad 1: +3V3 -> +1V2
- C16 pad 2: SLOT2SZ0 -> GND
- C17 pad 1: SLOT2SZ0 -> +3V3
- C17 pad 2: +3V3 -> GND
- C18 pad 1: SLOT2SZ0 -> +3V3
- C18 pad 2: +3V3 -> GND
- C19 pad 1: SLOT2SZ0 -> +3V3
- C19 pad 2: +3V3 -> GND
- C22 pad 2: SLOT2SZ0 -> GND
- C23 pad 2: SLOT2SZ0 -> GND
- C24 pad 1: SLOT2SZ0 -> GND
- C25 pad 1: +5V -> +1V2
- C25 pad 2: SLOT2SZ0 -> GND
- C26 pad 1: SLOT2SZ0 -> GND
- C28 pad 1: +5V -> +3V3
- C28 pad 2: SLOT2SZ0 -> GND
- C29 pad 2: SLOT2SZ0 -> GND
- C3 pad 1: SLOT2SZ0 -> GND
- C30 pad 1: SLOT2SZ0 -> GND
- C31 pad 1: SLOT2SZ0 -> GND
- C32 pad 1: SLOT2SZ0 -> GND
- C33 pad 1: SLOT2SZ0 -> GND
- C34 pad 2: SLOT2SZ0 -> GND
- C36 pad 1: +3V3 -> GND
- C36 pad 2: SLOT2SZ0 -> +3V3
- C37 pad 2: SLOT2SZ0 -> GND
- C38 pad 1: SLOT2SZ0 -> GND
- C39 pad 1: SLOT2SZ0 -> GND
- C4 pad 2: SLOT2SZ0 -> GND
- C40 pad 2: SLOT2SZ0 -> GND
- C41 pad 2: SLOT2SZ0 -> GND
- C42 pad 2: SLOT2SZ0 -> GND
- C43 pad 2: SLOT2SZ0 -> GND
- C44 pad 1: SLOT2SZ0 -> GND
- C45 pad 2: SLOT2SZ0 -> GND
- C47 pad 1: +1V2 -> +5V
- C47 pad 2: SLOT2SZ0 -> GND
- C48 pad 1: SLOT2SZ0 -> GND
- C49 pad 2: SLOT2SZ0 -> GND
- C5 pad 2: SLOT2SZ0 -> GND
- C50 pad 1: +1V2 -> +3V3
- C50 pad 2: SLOT2SZ0 -> GND
- C52 pad 2: SLOT2SZ0 -> GND
- C53 pad 1: +3V3 -> GND
- C53 pad 2: SLOT2SZ0 -> +3V3
- C54 pad 2: SLOT2SZ0 -> GND
- C55 pad 1: +5V -> +3V3
- C55 pad 2: SLOT2SZ0 -> GND
- C56 pad 2: SLOT2SZ0 -> GND
- C57 pad 2: SLOT2SZ0 -> GND
- C58 pad 1: +1V2 -> +3V3
- C58 pad 2: SLOT2SZ0 -> GND
- C59 pad 2: SLOT2SZ0 -> GND
- C6 pad 2: SLOT2SZ0 -> GND
- C60 pad 2: SLOT2SZ0 -> GND
- C61 pad 2: SLOT2SZ0 -> GND
- C62 pad 1: +1V2 -> +5V
- C62 pad 2: SLOT2SZ0 -> GND
- C63 pad 1: +3V3 -> +5V
- C63 pad 2: SLOT2SZ0 -> GND
- C64 pad 1: +1V2 -> +3V3
- C64 pad 2: SLOT2SZ0 -> GND
- C65 pad 1: +1V2 -> +3V3
- C65 pad 2: SLOT2SZ0 -> GND
- C66 pad 1: +3V3 -> +1V2
- C66 pad 2: SLOT2SZ0 -> GND
- C67 pad 1: +3V3 -> +1V2
- C67 pad 2: SLOT2SZ0 -> GND
- C68 pad 1: SLOT2SZ0 -> GND
- C69 pad 1: SLOT2SZ0 -> GND
- C7 pad 1: +3V3 -> GND
- C7 pad 2: SLOT2SZ0 -> +3V3
- C76 pad 2: SLOT2SZ0 -> GND
- C77 pad 2: SLOT2SZ0 -> GND
- C8 pad 2: SLOT2SZ0 -> GND
- C9 pad 1: +3V3 -> GND
- C9 pad 2: SLOT2SZ0 -> +3V3
- D7 pad 2: SLOT2SZ0 -> GND
- D9 pad 2: SLOT2SZ0 -> GND
- IC1 pad 4: SLOT2SZ0 -> GND
- IC19 pad 1: SLOT2SZ0 -> GND
- IC19 pad 10: A2 -> /MPU/A2
- IC19 pad 11: A3 -> /MPU/A3
- IC19 pad 12: A4 -> /MPU/A4
- IC19 pad 33: SLOT2SZ0 -> GND
- IC19 pad 36: SLOT2SZ0 -> GND
- IC19 pad 38: SLOT2SZ0 -> GND
- IC19 pad 39: SLOT2SZ0 -> GND
- IC19 pad 5: SLOT2SZ0 -> GND
- IC19 pad 6: SLOT2SZ0 -> GND
- IC24 pad 1: SLOT2SZ0 -> GND
- IC24 pad 10: SLOT2SZ0 -> GND
- IC24 pad 19: SLOT2SZ0 -> GND
- IC31 pad 1: Net-(IC33-E2) -> (no net)
- IC31 pad 11: E -> (no net)
- IC31 pad 12: S2 -> (no net)
- IC31 pad 13: Net-(IC33-E1) -> (no net)
- IC31 pad 2: R/~{W} -> (no net)
- IC31 pad 3: S2 -> (no net)
- IC31 pad 4: ~{R}/W -> (no net)
- IC31 pad 5: R/~{W} -> (no net)
- IC31 pad 6: R/~{W} -> (no net)
- IC31 pad 7: SLOT2SZ0 -> GND
- IC34 pad 8: SLOT2SZ0 -> GND
- J1 pad 5: SLOT2SZ0 -> GND
- J2 pad 4: SLOT2SZ0 -> GND
- J4 pad 2: SLOT2SZ0 -> GND
- J6 pad 17: SLOT2SZ0 -> GND
- J6 pad 2: SLOT2SZ0 -> GND
- J6 pad 20: SLOT2SZ0 -> GND
- J7 pad 17: SLOT2SZ0 -> GND
- J7 pad 2: SLOT2SZ0 -> GND
- J7 pad 20: SLOT2SZ0 -> GND
- J8 pad 2: SLOT2SZ0 -> GND
- JP1 pad 1: Z22 -> +3V3
- JP1 pad 2: Net-(JP1-B) -> /SAM/SZ0
- JP4 pad 2: SLOT2SZ0 -> GND
- PL1 pad 5: SLOT2SZ0 -> GND
- PL2 pad 10: SLOT2SZ0 -> GND
- PL2 pad 12: SLOT2SZ0 -> GND
- PL2 pad 14: SLOT2SZ0 -> GND
- PL2 pad 16: SLOT2SZ0 -> GND
- PL2 pad 18: SLOT2SZ0 -> GND
- PL2 pad 6: SLOT2SZ0 -> GND
- PL2 pad 8: SLOT2SZ0 -> GND
- PL3 pad 3: SLOT2SZ0 -> GND
- PL4 pad 2: SLOT2SZ0 -> GND
- PL5 pad 3: SLOT2SZ0 -> GND
- PL6 pad 5: SLOT2SZ0 -> GND
- PL6 pad 6: SLOT2SZ0 -> GND
- PL7 pad 33: SLOT2SZ0 -> GND
- PL7 pad 34: SLOT2SZ0 -> GND
- PL7 pad 4: ~{NMI} -> ~{NMIx}
- PL8 pad 33: SLOT2SZ0 -> GND
- PL8 pad 34: SLOT2SZ0 -> GND
- PL8 pad 4: ~{NMI} -> ~{NMIx}
- PL9 pad 1: SLOT2SZ0 -> GND
- R16 pad 1: SLOT2SZ0 -> GND
- R30 pad 1: SLOT2SZ0 -> GND
- R46 pad 1: SLOT2SZ0 -> GND
- R48 pad 1: SLOT2SZ0 -> GND
- R6 pad 1: ~{RAS0} -> SLOT2SZ0
- R6 pad 2: Net-(U18D-IO_L37N_3) -> GND
- R68 pad 1: SLOT2SZ0 -> GND
- R7 pad 1: ~{WE} -> +3V3
- R7 pad 2: Net-(U18D-IO_L42P_GCLK25_TRDY2_3) -> Net-(U18C-PROGRAM_B_2)
- R75 pad 1: SLOT2SZ0 -> GND
- R8 pad 1: +3V3 -> Net-(D10-K)
- R8 pad 2: Net-(U18C-PROGRAM_B_2) -> Net-(U18C-DONE_2)
- R9 pad 1: Net-(D10-K) -> EXTMEN
- R9 pad 2: Net-(U18C-DONE_2) -> +5V
- RN4 pad 10: Z22 -> Z1
- RN4 pad 11: Z21 -> Z0
- RN4 pad 6: /SAM/zZ21 -> /SAM/zZ0
- RN4 pad 7: /SAM/zZ22 -> /SAM/zZ1
- RN5 pad 1: /SAM/zZ0 -> /SAM/zZ2
- RN5 pad 10: Z6 -> Z8
- RN5 pad 11: Z5 -> Z7
- RN5 pad 12: Z4 -> Z6
- RN5 pad 13: Z3 -> Z5
- RN5 pad 14: Z2 -> Z4
- RN5 pad 15: Z1 -> Z3
- RN5 pad 16: Z0 -> Z2
- RN5 pad 2: /SAM/zZ1 -> /SAM/zZ3
- RN5 pad 3: /SAM/zZ2 -> /SAM/zZ4
- RN5 pad 4: /SAM/zZ3 -> /SAM/zZ5
- RN5 pad 5: /SAM/zZ4 -> /SAM/zZ6
- RN5 pad 6: /SAM/zZ5 -> /SAM/zZ7
- RN5 pad 7: /SAM/zZ6 -> /SAM/zZ8
- RN5 pad 8: /SAM/zZ7 -> /SAM/zZ9
- RN5 pad 9: Z7 -> Z9
- RN6 pad 1: /SAM/zZ8 -> /SAM/zZ10
- RN6 pad 14: Z10 -> Z21
- RN6 pad 15: Z9 -> Z22
- RN6 pad 16: Z8 -> Z10
- RN6 pad 2: /SAM/zZ9 -> /SAM/zZ22
- RN6 pad 3: /SAM/zZ10 -> /SAM/zZ21
- SW1 pad 2: SLOT2SZ0 -> GND
- SW1 pad 5: SLOT2SZ0 -> GND
- TR1 pad 3: SLOT2SZ0 -> GND
- U1 pad 11: SLOT2SZ0 -> GND
- U10 pad 4: SLOT2SZ0 -> GND
- U10 pad 6: SLOT2SZ0 -> GND
- U10 pad 7: SLOT2SZ0 -> GND
- U10 pad 8: SLOT2SZ0 -> GND
- U11 pad 3: SLOT2SZ0 -> GND
- U12 pad 1: SLOT2SZ0 -> GND
- U12 pad 16: SLOT2SZ0 -> GND
- U12 pad 17: SLOT2SZ0 -> GND
- U12 pad 26: ~{IRQ} -> ~{IRQx}
- U13 pad 1: Z20 -> Z19
- U13 pad 10: Z11 -> Z21
- U13 pad 11: R/~{W} -> RAM_R/~{W}
- U13 pad 13: Net-(JP1-B) -> Z22
- U13 pad 2: Z19 -> Z18
- U13 pad 25: Z1 -> Z0
- U13 pad 26: SLOT2SZ0 -> GND
- U13 pad 27: SLOT2SZ0 -> GND
- U13 pad 28: ~{R}/W -> RAM_~{OE}
- U13 pad 3: Z18 -> Z17
- U13 pad 4: Z17 -> Z16
- U13 pad 45: Z0 -> Z1
- U13 pad 46: SLOT2SZ0 -> GND
- U13 pad 47: SLOT2SZ0 -> GND
- U13 pad 48: Z21 -> Z20
- U13 pad 5: Z16 -> Z15
- U13 pad 6: Z15 -> Z14
- U13 pad 7: Z14 -> Z13
- U13 pad 8: Z13 -> Z12
- U13 pad 9: Z12 -> Z11
- U14 pad 3: SLOT2SZ0 -> GND
- U16 pad 1: /SAM/zA0 -> /SAM/zA7
- U16 pad 11: SLOT2SZ0 -> GND
- U16 pad 12: /MPU/A7 -> /MPU/A0
- U16 pad 13: /MPU/A6 -> /MPU/A1
- U16 pad 14: /MPU/A5 -> /MPU/A2
- U16 pad 15: A4 -> /MPU/A3
- U16 pad 16: A3 -> /MPU/A4
- U16 pad 17: A2 -> /MPU/A5
- U16 pad 18: /MPU/A1 -> /MPU/A6
- U16 pad 20: /MPU/A0 -> /MPU/A7
- U16 pad 3: /SAM/zA1 -> /SAM/zA6
- U16 pad 4: /SAM/zA2 -> /SAM/zA5
- U16 pad 5: /SAM/zA3 -> /SAM/zA4
- U16 pad 6: /SAM/zA4 -> /SAM/zA3
- U16 pad 7: /SAM/zA5 -> /SAM/zA2
- U16 pad 8: /SAM/zA6 -> /SAM/zA1
- U16 pad 9: /SAM/zA7 -> /SAM/zA0
- U17 pad 7: SLOT2SZ0 -> GND
- U18 pad P1: /MPU/D2 -> /MPU/D0
- U18 pad P100: /SAM/zZ19 -> /SAM/zZ6
- U18 pad P101: /SAM/zZ20 -> /SAM/zZ5
- U18 pad P102: /SAM/zZ21 -> /SAM/zZ4
- U18 pad P104: /SAM/zZ22 -> /SAM/zZ3
- U18 pad P105: /SAM/zZ23 -> /SAM/zZ2
- U18 pad P108: SLOT2SZ0 -> GND
- U18 pad P111: unconnected-(U18A-IO_L66N_SCP0_0-PadP111) -> /SAM/zA8
- U18 pad P112: unconnected-(U18A-IO_L66P_SCP1_0-PadP112) -> /SAM/zA9
- U18 pad P113: SLOT2SZ0 -> GND
- U18 pad P114: unconnected-(U18A-IO_L65N_SCP2_0-PadP114) -> /SAM/zA10
- U18 pad P115: unconnected-(U18A-IO_L65P_SCP3_0-PadP115) -> /SAM/zA11
- U18 pad P116: unconnected-(U18A-IO_L64N_SCP4_0-PadP116) -> /SAM/zA12
- U18 pad P117: unconnected-(U18A-IO_L64P_SCP5_0-PadP117) -> /SAM/zA13
- U18 pad P120: unconnected-(U18A-IO_L62N_VREF_0-PadP120) -> RAM_R/~{W}
- U18 pad P13: SLOT2SZ0 -> GND
- U18 pad P130: SLOT2SZ0 -> GND
- U18 pad P136: SLOT2SZ0 -> GND
- U18 pad P139: S0 -> S2
- U18 pad P141: S2 -> S0
- U18 pad P16: SLOT2SZ0 -> SLOT4SZ0
- U18 pad P17: SLOT2SZ0 -> SLOT4SZ0
- U18 pad P25: SLOT2SZ0 -> GND
- U18 pad P3: SLOT2SZ0 -> GND
- U18 pad P34: unconnected-(U18D-IO_L1N_VREF_3-PadP34) -> ~{HALT}
- U18 pad P39: unconnected-(U18C-IO_L65P_INIT_B_2-PadP39) -> ~{E}
- U18 pad P43: ~{CPU_READ} -> CPU_READ
- U18 pad P49: SLOT2SZ0 -> GND
- U18 pad P5: /MPU/D0 -> /MPU/D2
- U18 pad P54: SLOT2SZ0 -> GND
- U18 pad P57: unconnected-(U18C-IO_L14N_D12_2-PadP57) -> /SAM/zRnW
- U18 pad P58: unconnected-(U18C-IO_L14P_D11_2-PadP58) -> /SAM/zRES
- U18 pad P59: unconnected-(U18C-IO_L13N_D10_2-PadP59) -> RAM_~{OE}
- U18 pad P64: /SAM/zRES -> unconnected-(U18C-IO_L3N_MOSI_CSI_B_MISO0_2-PadP64)
- U18 pad P66: /SAM/zRnW -> unconnected-(U18C-IO_L2N_CMPMOSI_2-PadP66)
- U18 pad P68: SLOT2SZ0 -> GND
- U18 pad P74: /SAM/zZ16 -> /SAM/zZ23
- U18 pad P75: /SAM/zZ15 -> /SAM/zZ1
- U18 pad P77: SLOT2SZ0 -> GND
- U18 pad P78: /SAM/zZ14 -> /SAM/zZ0
- U18 pad P79: /SAM/zZ13 -> /SAM/zZ20
- U18 pad P80: /SAM/zZ12 -> /SAM/zZ19
- U18 pad P81: /SAM/zZ11 -> /SAM/zZ18
- U18 pad P82: /SAM/zZ10 -> /SAM/zZ17
- U18 pad P83: /SAM/zZ9 -> /SAM/zZ16
- U18 pad P84: /SAM/zZ8 -> /SAM/zZ15
- U18 pad P85: /SAM/zZ7 -> /SAM/zZ14
- U18 pad P87: /SAM/zZ6 -> /SAM/zZ13
- U18 pad P88: /SAM/zZ5 -> /SAM/zZ12
- U18 pad P91: SLOT2SZ0 -> GND
- U18 pad P92: /SAM/zZ4 -> /SAM/zZ11
- U18 pad P93: /SAM/zZ3 -> /SAM/zZ21
- U18 pad P94: /SAM/zZ2 -> /SAM/zZ22
- U18 pad P95: /SAM/zZ1 -> /SAM/zZ10
- U18 pad P96: SLOT2SZ0 -> GND
- U18 pad P97: /SAM/zZ0 -> /SAM/zZ9
- U18 pad P98: /SAM/zZ17 -> /SAM/zZ8
- U18 pad P99: /SAM/zZ18 -> /SAM/zZ7
- U19 pad 2: SLOT2SZ0 -> GND
- U2 pad 1: /SAM/zA8 -> /SAM/zA15
- U2 pad 11: SLOT2SZ0 -> GND
- U2 pad 12: /MPU/A15 -> /MPU/A8
- U2 pad 13: /MPU/A14 -> /MPU/A9
- U2 pad 14: /MPU/A13 -> /MPU/A10
- U2 pad 15: /MPU/A12 -> /MPU/A11
- U2 pad 16: /MPU/A11 -> /MPU/A12
- U2 pad 17: /MPU/A10 -> /MPU/A13
- U2 pad 18: /MPU/A9 -> /MPU/A14
- U2 pad 20: /MPU/A8 -> /MPU/A15
- U2 pad 3: /SAM/zA9 -> /SAM/zA14
- U2 pad 4: /SAM/zA10 -> /SAM/zA13
- U2 pad 5: /SAM/zA11 -> /SAM/zA12
- U2 pad 6: /SAM/zA12 -> /SAM/zA11
- U2 pad 7: /SAM/zA13 -> /SAM/zA10
- U2 pad 8: /SAM/zA14 -> /SAM/zA9
- U2 pad 9: /SAM/zA15 -> /SAM/zA8
- U20 pad 2: SLOT2SZ0 -> GND
- U21 pad 1: /SAM/zNMI -> /SAM/zLIC
- U21 pad 11: SLOT2SZ0 -> GND
- U21 pad 14: LIC -> ~{NMIx}
- U21 pad 17: ~{FIRQx} -> ~{IRQx}
- U21 pad 18: ~{IRQx} -> ~{FIRQx}
- U21 pad 20: ~{NMIx} -> LIC
- U21 pad 3: /SAM/zIRQ -> /SAM/zFIRQ
- U21 pad 4: /SAM/zFIRQ -> /SAM/zIRQ
- U21 pad 7: /SAM/zLIC -> /SAM/zNMI
- U3 pad 16: SLOT2SZ0 -> GND
- U3 pad 22: SLOT2SZ0 -> GND
- U4 pad 2: SLOT2SZ0 -> GND
- U5 pad 1: SLOT2SZ0 -> GND
- U5 pad 41: ~{IRQ} -> ~{IRQx}
- U5 pad 42: ~{IRQ} -> ~{IRQx}
- U6 pad 1: SLOT2SZ0 -> GND
- U6 pad 41: ~{FIRQ} -> ~{FIRQx}
- U6 pad 42: ~{FIRQ} -> ~{FIRQx}
- U7 pad 15: SLOT2SZ0 -> GND
- U8 pad 10: SLOT2SZ0 -> GND
- U8 pad 19: SLOT2SZ0 -> GND
- U9 pad 10: SLOT2SZ0 -> GND
- U9 pad 19: SLOT2SZ0 -> GND
- X2 pad 3: SLOT2SZ0 -> GND
- X3 pad 2: SLOT2SZ0 -> GND
Routing:
- net E: track 0.00 -> 656.1 mm, vias 0 -> 16
- net R/~{W}: track 0.00 -> 606.8 mm, vias 0 -> 15
- net ~{RES}: track 0.00 -> 574.0 mm, vias 0 -> 8
- net VCLK: track 0.00 -> 464.7 mm, vias 0 -> 4
- net +12V: track 0.00 -> 412.6 mm, vias 0 -> 2
- net ESND: track 0.00 -> 409.3 mm, vias 0 -> 5
- net /AUDIO/DC6: track 0.00 -> 406.2 mm, vias 0 -> 10
- net /AUDIO/DC2: track 0.00 -> 403.2 mm, vias 0 -> 10
- net /AUDIO/DC0: track 0.00 -> 403.2 mm, vias 0 -> 9
- net /AUDIO/DC3: track 0.00 -> 397.9 mm, vias 0 -> 10
- net /AUDIO/DC5: track 0.00 -> 397.7 mm, vias 0 -> 10
- net /AUDIO/DC1: track 0.00 -> 396.9 mm, vias 0 -> 10
- net /AUDIO/DC4: track 0.00 -> 393.8 mm, vias 0 -> 10
- net /AUDIO/DC7: track 0.00 -> 391.6 mm, vias 0 -> 9
- net /MPU/D0: track 0.00 -> 344.1 mm, vias 0 -> 7
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- added copper zone on In2.Cu, net +5V
- added copper zone on B.Cu, net GND
- added copper zone on F.Cu, net GND
- added copper zone on In1.Cu, net GND
- removed copper zone on B.Cu, net +12V
- removed copper zone on B.Cu, net +5V
- removed copper zone on F.Cu, net +5V
- removed copper zone on B.Cu, net SLOT2SZ0
- removed copper zone on F.Cu, net SLOT2SZ0
Other:
- copper layers 2 -> 4
- board text added: "3V3 BUS"
- board text added: "5V BUS"
- board text added: "ADDRESS BUS"
- board text added: "AVMA"
- board text added: "BUSY"
- board text added: "LIC"
- board text added: "Proto 3"
- board text added: "SAMx by Ciaran Anscomb"
- board text added: "SAMx4+ extenstions by Julian Brown"
- board text added: "TSC"
- board text removed: "EXTAL"
- board text removed: "MRDY"
- board text removed: "Proto 2"
- board text removed: "SAMx4 by Ciaran Anscomb"
- board text removed: "XTAL"
- board text removed: "~{DMA}"
