File: sam.kicad_sch (KiCad schematic)
At the start: 33 parts, among them IC10 74ACT138, IC11 74ACT244N, IC16 74ACT244N, IC31 74ACT02, IC33 74ACT138N, J4 JTAG, U1 AS6C1008-TIN, U2 AS6C1008-55TIN, U3 XC95144XL-TQ100, U4 TPS7A2433DBVR, X1 14.31818MHz

Commit message: switch to fpga
Parts:
- removed C3, C5: 0.1uF, Capacitor_SMD:C_0805_2012Metric_Pad1.18x1.45mm_HandSolder, symbol Device:C_Small
- removed C6: 4.7uF, Capacitor_Tantalum_SMD:CP_EIA-3216-18_Kemet-A_Pad1.58x1.35mm_HandSolder, symbol Device:C_Polarized_Small
- removed IC11, IC16: 74ACT244N, Package_SO:SOIC-20W_7.5x12.8mm_P1.27mm, symbol 74xx:74LS244
- removed JP1: 32k/64k, Connector_PinHeader_2.54mm:PinHeader_1x03_P2.54mm_Vertical, symbol Jumper:Jumper_3_Bridged12
- removed R2, R20, R27, R4: 22R, Resistor_SMD:R_0805_2012Metric_Pad1.20x1.40mm_HandSolder, symbol Device:R_Small
- removed R5: 100R, Resistor_SMD:R_0805_2012Metric_Pad1.20x1.40mm_HandSolder, symbol Device:R_Small
- removed RN1, RN2: 22R, Package_SO:SOIC-16_3.9x9.9mm_P1.27mm, symbol Motorola PIA:R_Pack_Split
- removed U1: AS6C1008-TIN, Package_SO:TSOP-I-32_18.4x8mm_P0.5mm, symbol Motorola PIA:AS6C1008
- removed U2: AS6C1008-55TIN, Package_SO:TSOP-I-32_18.4x8mm_P0.5mm, symbol Motorola PIA:AS6C1008
- removed U3: XC95144XL-TQ100, Package_QFP:TQFP-100_14x14mm_P0.5mm, symbol CPLD_Xilinx:XC95144XL-TQ100
- removed X1: 14.31818MHz, Oscillator:Oscillator_SMD_ECS_2520MV-xxx-xx-4Pin_2.5x2.0mm, symbol Oscillator:ECS-2520MV-xxx-xx
- added C17: 100uF, Capacitor_SMD:C_0805_2012Metric, symbol Device:C_Small
- added C18, C19, C25, C28, C74, C75: 0.1uF, Capacitor_SMD:C_0805_2012Metric_Pad1.18x1.45mm_HandSolder, symbol Device:C_Small
- added C29, C34, C47, C49, C52, C53, C54, C56, C59, C64, C65, C66, C67, C70: 4.7uF, Capacitor_SMD:C_0805_2012Metric_Pad1.18x1.45mm_HandSolder, symbol Device:C_Small
- added C36, C37, C40, C41, C50, C57, C60, C71, C72, C73: 0.47uF, Capacitor_SMD:C_0805_2012Metric_Pad1.18x1.45mm_HandSolder, symbol Device:C_Small
- added C55, C58, C61, C62: 1u, Capacitor_SMD:C_0805_2012Metric_Pad1.18x1.45mm_HandSolder, symbol Device:C
- added C63: 0.01uF, Capacitor_SMD:C_0805_2012Metric_Pad1.18x1.45mm_HandSolder, symbol Device:C_Small
- added D10: LED_RED, LED_SMD:LED_0805_2012Metric, symbol Device:LED_Small
- added JP1: Enable 8M, Jumper:SolderJumper-2_P1.3mm_Open_Pad1.0x1.5mm, symbol Jumper:Jumper_2_Small_Open
- added R10, R11: 10K, Resistor_SMD:R_0805_2012Metric_Pad1.20x1.40mm_HandSolder, symbol Device:R
- added R6, R7: 22R, Resistor_SMD:R_0805_2012Metric_Pad1.20x1.40mm_HandSolder, symbol Device:R_Small
- added R8: 4K7, Resistor_SMD:R_0805_2012Metric_Pad1.20x1.40mm_HandSolder, symbol Device:R
- added R9: 1K, Resistor_SMD:R_0805_2012Metric_Pad1.20x1.40mm_HandSolder, symbol Device:R
- added RN4, RN5, RN6: 22R, Package_SO:SOIC-16W_5.3x10.2mm_P1.27mm, symbol Motorola PIA:R_Pack_Split
- added TP1: TP_VCLK, TestPoint:TestPoint_Loop_D1.80mm_Drill1.0mm_Beaded, symbol Connector:TestPoint_Flag
- added TP2: TP_DA0, TestPoint:TestPoint_Loop_D1.80mm_Drill1.0mm_Beaded, symbol Connector:TestPoint_Flag
- added TP3: TP_OSC, TestPoint:TestPoint_Loop_D1.80mm_Drill1.0mm_Beaded, symbol Connector:TestPoint_Flag
- added U13: RMLV3216A, Package_SO:TSOP-I-48_18.4x12mm_P0.5mm, symbol MemorySRAM:RMLV3216
- added U16, U2, U21: MAX3012, Package_SO:TSSOP-20_4.4x6.5mm_P0.65mm, symbol Motorola PIA:MAX3012
- added U18: XC6SLX9-2TQG144I, Dragon:AMD-LQFP-144, symbol 6847:XC6SLX9-3TQG144I
- added U19, U20: SN105125DBVR, Package_TO_SOT_SMD:SOT-23-5, symbol Regulator_Linear:TPS7A0533PDBV
- added X3: 14.31818MHz, Oscillator:Oscillator_SMD_ECS_2520MV-xxx-xx-4Pin_2.5x2.0mm, symbol Oscillator:ECS-2520MV-xxx-xx
- R3: value 22R -> 100R; DigiKey CF14JT22R0CT-ND -> RNCP0805FTD100RCT-ND
Connections:
- net ~{CAS} is gone; now on net VCLK: R3.1
- net +3V3: now also C17.2, C18.2, C19.2, C29.1, C34.1, C36.1, C37.1, C40.1, C41.1, C49.1, C52.1, C53.1, C54.1, C56.1, C57.1, C59.1, C60.1, C63.1, C66.1, C67.1, C70.1, C71.1, C72.1, C73.1, C74.2, D10.2 (A), R8.1, U13.12 (CS2), U13.37 (Vcc), U16.10 (EN), U16.2 (VL), U18.P103 (VCCO_1__2), U18.P122 (VCCO_0), U18.P125 (VCCO_0__1), U18.P129 (VCCAUX__4), U18.P135 (VCCO_0__2), U18.P18 (VCCO_3__1), U18.P20 (VCCAUX), U18.P31 (VCCO_3__2), U18.P36 (VCCAUX__1), U18.P4 (VCCO_3), U18.P42 (VCCO_2), U18.P53 (VCCAUX__2), U18.P63 (VCCO_2__1), U18.P76 (VCCO_1), U18.P86 (VCCO_1__1), U18.P90 (VCCAUX__3), U2.10 (EN), U2.2 (VL), U21.10 (EN), U21.2 (VL), X3.1 (Tri-State), X3.4 (VDD)
- net +5V: now also C25.1, C28.1, C55.1, C61.1, C75.1, U16.19 (VCC), U19.1 (IN), U19.3 (EN), U2.19 (VCC), U20.1 (IN), U20.3 (EN), U21.19 (VCC)
- net A0: now also U16.20 (VCC1)
- net A1: now also U16.18 (VCC2)
- net A10: now also U2.17 (VCC3)
- net A11: now also U2.16 (VCC4)
- net A12: now also U2.15 (VCC5)
- net A13: now also U2.14 (VCC6)
- net A14: now also U2.13 (VCC7)
- net A15: now also U2.12 (VCC8)
- net A2: now also U16.17 (VCC3)
- net A3: now also U16.16 (VCC4)
- net A4: now also U16.15 (VCC5)
- net A5: now also U16.14 (VCC6)
- net A6: now also U16.13 (VCC7)
- net A7: now also U16.12 (VCC8)
- net A8: now also U2.20 (VCC1)
- net A9: now also U2.18 (VCC2)
- net D0: now also U13.44 (DQ7), U18.P5 (IO_L52N_3)
- net D1: now also U13.42 (DQ6), U18.P2 (IO_L83P_3)
- net D2: now also U13.40 (DQ5), U18.P1 (IO_L83N_VREF_3)
- net D3: now also U13.38 (DQ4), U18.P6 (IO_L52P_3)
- net D4: now also U13.35 (DQ3), U18.P7 (IO_L51N_3)
- net D5: now also U13.33 (DQ2), U18.P8 (IO_L51P_3)
- net D6: now also U13.31 (DQ1), U18.P9 (IO_L50N_3)
- net D7: now also U13.29 (DQ0), U18.P10 (IO_L50P_3)
- net DA0: now also TP2.1, U18.P124 (IO_L37P_GCLK13_0)
- net E: now also U18.P24 (IO_L41P_GCLK27_3)
- net GND: now also C17.1, C18.1, C19.1, C25.2, C28.2, C29.2, C34.2, C36.2, C37.2, C40.2, C41.2, C47.2, C49.2, C50.2, C52.2, C53.2, C54.2, C55.2, C56.2, C57.2, C58.2, C59.2, C60.2, C61.2, C62.2, C63.2, C64.2, C65.2, C66.2, C67.2, C70.2, C71.2, C72.2, C73.2, C74.1, C75.2, U13.26 (~{CS1}), U13.27 (Vss), U13.46 (Vss), U13.47 (~{BYTE}), U16.11 (GND), U18.P108 (GND__9), U18.P11 (IO_L49N_3), U18.P113 (GND__10), U18.P12 (IO_L49P_3), U18.P13 (GND__1), U18.P130 (GND__11), U18.P136 (GND__12), U18.P14 (IO_L44N_GCLK20_3), U18.P15 (IO_L44P_GCLK21_3), U18.P16 (IO_L43N_GCLK22_IRDY2_3), U18.P17 (IO_L43P_GCLK23_3), U18.P25 (GND__2), U18.P3 (GND), U18.P49 (GND__3), U18.P54 (GND__4), U18.P68 (GND__5), U18.P77 (GND__6), U18.P91 (GND__7), U18.P96 (GND__8), U19.2 (GND), U2.11 (GND), U20.2 (GND), U21.11 (GND), X3.2 (GND)
- net OSC: now also TP3.1, U18.P123 (IO_L37N_GCLK12_0), X3.3 (OUT)
- net Q: now also U18.P23 (IO_L41N_GCLK26_3)
- net R/~{W}: now also U13.11 (~{WE}), U21.16 (VCC4)
- net S0: now also U18.P139 (IO_L3N_0)
- net S1: now also U18.P140 (IO_L3P_0)
- net S2: now also U18.P141 (IO_L2N_0)
- net TCK: now also U18.P109 (TCK)
- net TDI0: now also U18.P106 (TDO)
- net TDI1: now also U18.P110 (TDI)
- net TMS: now also U18.P107 (TMS)
- net VCLK: now also TP1.1
- net Z0: now also RN5.16, U13.45 (DQ15/A-1)
- net Z1: now also RN5.15, U13.25 (A0)
- net Z10: now also RN6.14, U13.16 (A18)
- net Z11: now also RN6.13, U13.10 (A20)
- net Z12: now also RN6.12, U13.9 (A19)
- net Z13: now also RN6.11, U13.8 (A8)
- net Z14: now also RN6.10, U13.7 (A9)
- net Z15: now also RN6.9, U13.6 (A10)
- net Z16: now also RN4.16, U13.5 (A11)
- net Z17: now also RN4.15, U13.4 (A12)
- net Z2: now also RN5.14, U13.24 (A1)
- net Z3: now also RN5.13, U13.23 (A2)
- net Z4: now also RN5.12, U13.22 (A3)
- net Z5: now also RN5.11, U13.21 (A4)
- net Z6: now also RN5.10, U13.20 (A5)
- net Z7: now also RN5.9, U13.19 (A6)
- net Z8: now also RN6.16, U13.18 (A7)
- net Z9: now also RN6.15, U13.17 (A17)
- net ~{NHS}: now also U18.P65 (IO_L3P_D0_DIN_MISO_MISO1_2)
- net ~{RAS0}: now also R6.1
- net ~{R}/W: now also U13.28 (~{OE})
- net ~{WE}: now also R7.1
- net at IC33.5 (E2): now also IC31.1
- net at R3.2: now also U18.P35 (IO_L1P_3)
- new net: R11.1, U20.4 (POK)
- new net: R7.2, U18.P22 (IO_L42P_GCLK25_TRDY2_3)
- new net: R6.2, U18.P26 (IO_L37N_3)
- new net: R10.1, U19.4 (POK)
- new net: JP1.2 (B), U13.13 (NC)
- new net: R8.2, U18.P37 (PROGRAM_B_2)
- new net: D10.1 (K), R9.1
- new net: R9.2, U18.P71 (DONE_2)
- new net +1V2: C47.1, C50.1, C58.1, C62.1, C64.1, C65.1, R10.2, R11.2, U18.P128 (VCCINT__4), U18.P19 (VCCINT), U18.P28 (VCCINT__1), U18.P52 (VCCINT__2), U18.P89 (VCCINT__3), U19.5 (OUT), U20.5 (OUT)
- new net LIC: U21.14 (VCC6)
- new net SZ0: U18.P67 (IO_L2P_CMPCLK_2)
- new net SZ1: U18.P69 (IO_L1N_M0_CMPMISO_2)
- new net SZ2: U18.P70 (IO_L1P_CCLK_2)
- new net Z18: RN4.14, U13.3 (A13)
- new net Z19: RN4.13, U13.2 (A14)
- new net Z20: RN4.12, U13.1 (A15)
- new net Z21: RN4.11, U13.48 (A16)
- new net Z22: JP1.1 (A), RN4.10
- new net Z23: RN4.9
- new net zA0: U16.1 (VL1), U18.P126 (IO_L36N_GCLK14_0)
- new net zA1: U16.3 (VL2), U18.P127 (IO_L36P_GCLK15_0)
- new net zA10: U2.4 (VL3)
- new net zA11: U2.5 (VL4)
- new net zA12: U2.6 (VL5)
- new net zA13: U2.7 (VL6)
- new net zA14: U18.P118 (IO_L63N_SCP6_0), U2.8 (VL7)
- new net zA15: U18.P119 (IO_L63P_SCP7_0), U2.9 (VL8)
- new net zA2: U16.4 (VL3), U18.P131 (IO_L35N_GCLK16_0)
- new net zA3: U16.5 (VL4), U18.P132 (IO_L35P_GCLK17_0)
- new net zA4: U16.6 (VL5), U18.P133 (IO_L34N_GCLK18_0)
- new net zA5: U16.7 (VL6), U18.P134 (IO_L34P_GCLK19_0)
- new net zA6: U16.8 (VL7), U18.P137 (IO_L4N_0)
- new net zA7: U16.9 (VL8), U18.P138 (IO_L4P_0)
- new net zA8: U2.1 (VL1)
- new net zA9: U2.3 (VL2)
- new net zFIRQ: U18.P47 (IO_L48N_RDWR_B_VREF_2), U21.4 (VL3)
- new net zIRQ: U18.P46 (IO_L49P_D3_2), U21.3 (VL2)
- new net zLIC: U18.P48 (IO_L48P_D7_2), U21.7 (VL6)
- new net zNMI: U18.P45 (IO_L49N_D4_2), U21.1 (VL1)
- new net zRES: U18.P64 (IO_L3N_MOSI_CSI_B_MISO0_2), U21.6 (VL5)
- new net zRnW: U18.P66 (IO_L2N_CMPMOSI_2), U21.5 (VL4)
- new net zZ0: RN5.1, U18.P97 (IO_L34N_1)
- new net zZ1: RN5.2, U18.P95 (IO_L40P_GCLK11_1)
- new net zZ10: RN6.3, U18.P82 (IO_L45N_1)
- new net zZ11: RN6.4, U18.P81 (IO_L46P_1)
- new net zZ12: RN6.5, U18.P80 (IO_L46N_1)
- new net zZ13: RN6.6, U18.P79 (IO_L47P_1)
- new net zZ14: RN6.7, U18.P78 (IO_L47N_1)
- new net zZ15: RN6.8, U18.P75 (IO_L74P_AWAKE_1)
- new net zZ16: RN4.1, U18.P74 (IO_L74N_DOUT_BUSY_1)
- new net zZ17: RN4.2, U18.P98 (IO_L34P_1)
- new net zZ18: RN4.3, U18.P99 (IO_L33N_1)
- new net zZ19: RN4.4, U18.P100 (IO_L33P_1)
- new net zZ2: RN5.3, U18.P94 (IO_L40N_GCLK10_1)
- new net zZ20: RN4.5, U18.P101 (IO_L32N_1)
- new net zZ21: RN4.6, U18.P102 (IO_L32P_1)
- new net zZ22: RN4.7, U18.P104 (IO_L1N_VREF_1)
- new net zZ23: RN4.8, U18.P105 (IO_L1P_1)
- new net zZ3: RN5.4, U18.P93 (IO_L41P_GCLK9_IRDY1_1)
- new net zZ4: RN5.5, U18.P92 (IO_L41N_GCLK8_1)
- new net zZ5: RN5.6, U18.P88 (IO_L42P_GCLK7_1)
- new net zZ6: RN5.7, U18.P87 (IO_L42N_GCLK6_TRDY1_1)
- new net zZ7: RN5.8, U18.P85 (IO_L43P_GCLK5_1)
- new net zZ8: RN6.1, U18.P84 (IO_L43N_GCLK4_1)
- new net zZ9: RN6.2, U18.P83 (IO_L45P_1)
- new net ~{CPU_ACTIVE}: U18.P40 (IO_L64N_D9_2)
- new net ~{CPU_READ}: U18.P43 (IO_L62N_D6_2)
- new net ~{CPU_WRITE}: U18.P44 (IO_L62P_D5_2)
- new net ~{FIRQx}: U21.17 (VCC3)
- new net ~{FIRQ}: U18.P60 (IO_L13P_M1_2)
- new net ~{IRQx}: U21.18 (VCC2)
- new net ~{IRQ}: U18.P61 (IO_L12N_D2_MISO3_2)
- new net ~{NMIx}: U21.20 (VCC1)
- new net ~{NMI}: U18.P62 (IO_L12P_D1_MISO2_2)
- new net ~{RES}: U21.15 (VCC5)
- no-connect marks 2 -> 34
Other:
- moved on the sheet: IC10, IC31A, IC31B, IC31D, IC33, R39

Commit message: rework traces for FPGA
Parts:
- removed C11, C12, C13, C14, C15, C16: 100n, Capacitor_SMD:C_0805_2012Metric_Pad1.18x1.45mm_HandSolder, symbol Device:C
- removed JP1: Enable 8M, Jumper:SolderJumper-2_P1.3mm_Open_Pad1.0x1.5mm, symbol Jumper:Jumper_2_Small_Open
- added unit 3 of IC2
- added JP1: SZ0, Jumper:SolderJumper-2_P1.3mm_Bridged_Pad1.0x1.5mm, symbol Jumper:Jumper_2_Small_Bridged
- added JP6: SZ1, Jumper:SolderJumper-2_P1.3mm_Open_Pad1.0x1.5mm, symbol Jumper:Jumper_2_Small_Open
- added JP7: SZ2, Jumper:SolderJumper-2_P1.3mm_Bridged_Pad1.0x1.5mm, symbol Jumper:Jumper_2_Small_Bridged
- added R12, R13, R14, R2, R6: 4K7, Resistor_SMD:R_0805_2012Metric_Pad1.20x1.40mm_HandSolder, symbol Device:R
- C53: renamed from C17; footprint Capacitor_SMD:C_0805_2012Metric -> Capacitor_SMD:C_0805_2012Metric_Pad1.18x1.45mm_HandSolder
- renumbered C28 to C11, C47 to C12, C49 to C13, C64 to C14, C66 to C15, C65 to C16, C67 to C17, C29 to C18, C34 to C19, C50 to C25, C52 to C28, C36 to C29, C37 to C34, C74 to C36, C53 to C37, C75 to C47, C54 to C49, C56 to C50, C57 to C52, C70 to C54, C59 to C55, C71 to C56, C72 to C57, C60 to C58, C73 to C59, C63 to C60, C55 to C61, C61 to C62, C8 to C63, C9 to C64, C7 to C65, C58 to C66, C62 to C67, C18 to C7, C25 to C8, C19 to C9, IC31 to IC2, IC33 to IC3, IC10 to IC4, R6 to R4, R7 to R5, R8 to R7, R9 to R8, R39 to R9, RN6 to RN4, RN4 to RN6
Connections:
- net +3V3: now also JP1.1 (A), JP6.1 (A), JP7.1 (A)
- net A0: now also U16.12 (VCC8); no longer U16.20 (VCC1)
- net A1: now also U16.13 (VCC7); no longer U16.18 (VCC2)
- net A10: now also U2.14 (VCC6); no longer U2.17 (VCC3)
- net A11: now also U2.15 (VCC5); no longer U2.16 (VCC4)
- net A12: now also U2.16 (VCC4); no longer U2.15 (VCC5)
- net A13: now also U2.17 (VCC3); no longer U2.14 (VCC6)
- net A14: now also U2.18 (VCC2); no longer U2.13 (VCC7)
- net A15: now also U2.20 (VCC1); no longer U2.12 (VCC8)
- net A2: now also U16.14 (VCC6); no longer IC4.1 (A0), U16.17 (VCC3)
- net A3: now also U16.15 (VCC5); no longer IC4.2 (A1), U16.16 (VCC4)
- net A4: now also U16.16 (VCC4); no longer IC4.3 (A2), U16.15 (VCC5)
- net A5: now also U16.17 (VCC3); no longer U16.14 (VCC6)
- net A6: now also U16.18 (VCC2); no longer U16.13 (VCC7)
- net A7: now also U16.20 (VCC1); no longer U16.12 (VCC8)
- net A8: now also U2.12 (VCC8); no longer U2.20 (VCC1)
- net A9: now also U2.13 (VCC7); no longer U2.18 (VCC2)
- net D0: now also U18.P1 (IO_L83N_VREF_3); no longer U18.P5 (IO_L52N_3)
- net D2: now also U18.P5 (IO_L52N_3); no longer U18.P1 (IO_L83N_VREF_3)
- net GND: now also R12.2, R13.2, R14.2, R2.1, R6.2; no longer U18.P11 (IO_L49N_3), U18.P12 (IO_L49P_3), U18.P14 (IO_L44N_GCLK20_3), U18.P15 (IO_L44P_GCLK21_3), U18.P16 (IO_L43N_GCLK22_IRDY2_3), U18.P17 (IO_L43P_GCLK23_3)
- net LIC: now also U21.20 (VCC1); no longer U21.14 (VCC6)
- net R/~{W}: no longer IC2.5, IC2.6, U13.11 (~{WE})
- net S0: now also U18.P141 (IO_L2N_0); no longer U18.P139 (IO_L3N_0)
- net S2: now also U18.P139 (IO_L3N_0); no longer U18.P141 (IO_L2N_0)
- net SZ0: now also JP1.2 (B), R12.1
- net SZ1: now also JP6.2 (B), R13.1
- net SZ2: now also JP7.2 (B), R14.1
- net Z0: now also RN4.11, U13.25 (A0); no longer RN5.16, U13.45 (DQ15/A-1)
- net Z1: now also RN4.10, U13.45 (DQ15/A-1); no longer RN5.15, U13.25 (A0)
- net Z10: now also RN6.16; no longer RN6.14
- net Z11: now also U13.9 (A19); no longer U13.10 (A20)
- net Z12: now also U13.8 (A8); no longer U13.9 (A19)
- net Z13: now also U13.7 (A9); no longer U13.8 (A8)
- net Z14: now also U13.6 (A10); no longer U13.7 (A9)
- net Z15: now also U13.5 (A11); no longer U13.6 (A10)
- net Z16: now also RN4.16, U13.4 (A12); no longer RN4.16, U13.5 (A11)
- net Z17: now also RN4.15, U13.3 (A13); no longer RN4.15, U13.4 (A12)
- net Z18: now also U13.2 (A14); no longer U13.3 (A13)
- net Z19: now also U13.1 (A15); no longer U13.2 (A14)
- net Z2: now also IC4.1 (A0), RN5.16; no longer RN5.14
- net Z20: now also U13.48 (A16); no longer U13.1 (A15)
- net Z21: now also RN6.14, U13.10 (A20); no longer RN6.11, U13.48 (A16)
- net Z22: now also RN6.15, U13.13 (NC); no longer RN6.10
- net Z3: now also IC4.2 (A1), RN5.15; no longer RN5.13
- net Z4: now also IC4.3 (A2), RN5.14; no longer RN5.12
- net Z5: now also RN5.13; no longer RN5.11
- net Z6: now also RN5.12; no longer RN5.10
- net Z7: now also RN5.11; no longer RN5.9
- net Z8: now also RN5.10; no longer RN4.16
- net Z9: now also RN5.9; no longer RN4.15
- net zA0: now also U16.9 (VL8); no longer U16.1 (VL1)
- net zA1: now also U16.8 (VL7); no longer U16.3 (VL2)
- net zA10: now also U18.P114 (IO_L65N_SCP2_0), U2.7 (VL6); no longer U2.4 (VL3)
- net zA11: now also U18.P115 (IO_L65P_SCP3_0), U2.6 (VL5); no longer U2.5 (VL4)
- net zA12: now also U18.P116 (IO_L64N_SCP4_0), U2.5 (VL4); no longer U2.6 (VL5)
- net zA13: now also U18.P117 (IO_L64P_SCP5_0), U2.4 (VL3); no longer U2.7 (VL6)
- net zA14: now also U2.3 (VL2); no longer U2.8 (VL7)
- net zA15: now also U2.1 (VL1); no longer U2.9 (VL8)
- net zA2: now also U16.7 (VL6); no longer U16.4 (VL3)
- net zA3: now also U16.6 (VL5); no longer U16.5 (VL4)
- net zA4: now also U16.5 (VL4); no longer U16.6 (VL5)
- net zA5: now also U16.4 (VL3); no longer U16.7 (VL6)
- net zA6: now also U16.3 (VL2); no longer U16.8 (VL7)
- net zA7: now also U16.1 (VL1); no longer U16.9 (VL8)
- net zA8: now also U18.P111 (IO_L66N_SCP0_0), U2.9 (VL8); no longer U2.1 (VL1)
- net zA9: now also U18.P112 (IO_L66P_SCP1_0), U2.8 (VL7); no longer U2.3 (VL2)
- net zFIRQ: now also U21.3 (VL2); no longer U21.4 (VL3)
- net zIRQ: now also U21.4 (VL3); no longer U21.3 (VL2)
- net zLIC: now also U21.1 (VL1); no longer U21.7 (VL6)
- net zNMI: now also U21.7 (VL6); no longer U21.1 (VL1)
- net zRES: now also U18.P58 (IO_L14P_D11_2); no longer U18.P64 (IO_L3N_MOSI_CSI_B_MISO0_2)
- net zRnW: now also U18.P57 (IO_L14N_D12_2); no longer U18.P66 (IO_L2N_CMPMOSI_2)
- net zZ0: now also RN4.6, U18.P78 (IO_L47N_1); no longer RN5.1, U18.P97 (IO_L34N_1)
- net zZ1: now also RN4.7, U18.P75 (IO_L74P_AWAKE_1); no longer RN5.2, U18.P95 (IO_L40P_GCLK11_1)
- net zZ10: now also RN6.1, U18.P95 (IO_L40P_GCLK11_1); no longer RN6.3, U18.P82 (IO_L45N_1)
- net zZ11: now also U18.P92 (IO_L41N_GCLK8_1); no longer U18.P81 (IO_L46P_1)
- net zZ12: now also U18.P88 (IO_L42P_GCLK7_1); no longer U18.P80 (IO_L46N_1)
- net zZ13: now also U18.P87 (IO_L42N_GCLK6_TRDY1_1); no longer U18.P79 (IO_L47P_1)
- net zZ14: now also U18.P85 (IO_L43P_GCLK5_1); no longer U18.P78 (IO_L47N_1)
- net zZ15: now also U18.P84 (IO_L43N_GCLK4_1); no longer U18.P75 (IO_L74P_AWAKE_1)
- net zZ16: now also RN4.1, U18.P83 (IO_L45P_1); no longer RN4.1, U18.P74 (IO_L74N_DOUT_BUSY_1)
- net zZ17: now also RN4.2, U18.P82 (IO_L45N_1); no longer RN4.2, U18.P98 (IO_L34P_1)
- net zZ18: now also U18.P81 (IO_L46P_1); no longer U18.P99 (IO_L33N_1)
- net zZ19: now also U18.P80 (IO_L46N_1); no longer U18.P100 (IO_L33P_1)
- net zZ2: now also RN5.1, U18.P105 (IO_L1P_1); no longer RN5.3, U18.P94 (IO_L40N_GCLK10_1)
- net zZ20: now also U18.P79 (IO_L47P_1); no longer U18.P101 (IO_L32N_1)
- net zZ21: now also RN6.3, U18.P93 (IO_L41P_GCLK9_IRDY1_1); no longer RN6.6, U18.P102 (IO_L32P_1)
- net zZ22: now also RN6.2, U18.P94 (IO_L40N_GCLK10_1); no longer RN6.7, U18.P104 (IO_L1N_VREF_1)
- net zZ23: now also U18.P74 (IO_L74N_DOUT_BUSY_1); no longer U18.P105 (IO_L1P_1)
- net zZ3: now also RN5.2, U18.P104 (IO_L1N_VREF_1); no longer RN5.4, U18.P93 (IO_L41P_GCLK9_IRDY1_1)
- net zZ4: now also RN5.3, U18.P102 (IO_L32P_1); no longer RN5.5, U18.P92 (IO_L41N_GCLK8_1)
- net zZ5: now also RN5.4, U18.P101 (IO_L32N_1); no longer RN5.6, U18.P88 (IO_L42P_GCLK7_1)
- net zZ6: now also RN5.5, U18.P100 (IO_L33P_1); no longer RN5.7, U18.P87 (IO_L42N_GCLK6_TRDY1_1)
- net zZ7: now also RN5.6, U18.P99 (IO_L33N_1); no longer RN5.8, U18.P85 (IO_L43P_GCLK5_1)
- net zZ8: now also RN5.7, U18.P98 (IO_L34P_1); no longer RN4.1, U18.P84 (IO_L43N_GCLK4_1)
- net zZ9: now also RN5.8, U18.P97 (IO_L34N_1); no longer RN4.2, U18.P83 (IO_L45P_1)
- net ~{FIRQx}: now also U21.18 (VCC2); no longer U21.17 (VCC3)
- net ~{IRQx}: now also U21.17 (VCC3); no longer U21.18 (VCC2)
- net ~{NMIx}: now also U21.14 (VCC6); no longer U21.20 (VCC1)
- net ~{HALT}: now reaches U18.P34 (IO_L1N_VREF_3)
- net RAM_R/~{W}: now reaches U18.P120 (IO_L62N_VREF_0)
- net RAM_R/~{W}: now also U13.11 (~{WE})
- net ~{E}: now reaches U18.P39 (IO_L65P_INIT_B_2)
- net RAM_~{OE}: now reaches U18.P59 (IO_L13N_D10_2)
- net RAM_~{OE}: now also U13.28 (~{OE})
- net ~{CPU_READ} renamed CPU_READ
- net ~{CPU_WRITE} renamed CPU_WRITE
- net ~{R}/W: no longer names the net of IC2.4
- net ~{R}/W: no longer U13.28 (~{OE})
- new net SLOT2SZ0: R6.1, U18.P11 (IO_L49N_3), U18.P12 (IO_L49P_3), U18.P14 (IO_L44N_GCLK20_3), U18.P15 (IO_L44P_GCLK21_3)
- new net SLOT4SZ0: R2.2, U18.P16 (IO_L43N_GCLK22_IRDY2_3), U18.P17 (IO_L43P_GCLK23_3)
- no-connect marks 34 -> 40
Other:
- moved on the sheet: C62, C67, R11, RN4A, RN4B, RN4C, RN4D, RN4E, RN4F, RN4G, RN4H, RN5A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
